Commit message: 5 dof

File: koko_gazebo/robots/6dof_dyn2.urdf (robot description, URDF)
Before this commit: robot sixDOF_tracker_dyn_v11, 8 links, 7 joints
Links:
- link base_link: geometry collision mesh filename=package://koko_gazebo/meshes/base_link.STL; visual mesh filename=package://koko_gazebo/meshes/base_link.STL
- link elbow_link: geometry collision mesh filename=package://koko_gazebo/meshes/elbow_link.STL; visual mesh filename=package://koko_gazebo/meshes/elbow_link.STL
- link eroll_link: geometry collision mesh filename=package://koko_gazebo/meshes/eroll_link.STL; visual mesh filename=package://koko_gazebo/meshes/eroll_link.STL
- link lift_link: geometry collision mesh filename=package://koko_gazebo/meshes/lift_link.STL; visual mesh filename=package://koko_gazebo/meshes/lift_link.STL
- link sroll_link: geometry collision mesh filename=package://koko_gazebo/meshes/sroll_link.STL; visual mesh filename=package://koko_gazebo/meshes/sroll_link.STL
- link wrist_link: geometry collision mesh filename=package://koko_gazebo/meshes/wrist_link.STL; visual mesh filename=package://koko_gazebo/meshes/wrist_link.STL
- link wroll_link: geometry collision mesh filename=package://koko_gazebo/meshes/wroll_link.STL; visual mesh filename=package://koko_gazebo/meshes/wroll_link.STL
