Commit message: Added Cartesian Pose Controller

File: koko_descriptions/koko_description_sevendof_kin/robots/koko_description_sevendof_kin.urdf (robot description, URDF)
Before this commit: robot koko_description_sevendof_kin, 13 links, 12 joints
Links:
- link base_tracker_link: mass 0.0852031303342033 -> 0.0852031301907352
- link ee_tracker_link: mass 0.0852083037017581 -> 0.0852083038792347
- link forearm_link: mass 4.11546002120227 -> 4.11546002232608
- link forearm_tracker_link: mass 0.08520580160168 -> 0.0852058022688607
- link kinect_link: mass 0.813673516458148 -> 0.813673516453062
- link shoulder_lift_link: mass 0.437261383344081 -> 0.437261383344117
- link shoulder_link: mass 4.07268028424284 -> 4.07268991609326
- link upper_arm_lift_link: mass 0.42452313343894 -> 0.424523133438859
- link upper_arm_link: mass 4.1890717055091 -> 4.18907578737678
- link upper_arm_tracker_link: mass 0.0852060549513915 -> 0.0852060551384698
Joints:
- joint elbow_lift_joint: origin xyz=-0.0114299542278803 3.04774860032109E-05 0.181015691181535 rpy=-1.5707963267949 -0.355504877844586 -0.0026664457665753 -> xyz=-0.0114299548892374 3.04756154084207E-05 0.181015691851649 rpy=-1.5707963267949 -0.355504877844586 -0.0026664457665753
- joint elbow_roll_joint: origin xyz=0.00778446378216613 -0.0702248717036259 0 rpy=1.5707963267949 -0.00251502707069075 0.11039980475715 -> xyz=0.00778446477696024 -0.0702248702858572 0 rpy=1.5707963267949 -0.00251502707069075 0.11039980475715
- joint forearm_tracker_joint: origin xyz=0.0683718591042195 -0.000172162781444607 0.0965426884037958 rpy=1.26028779817361 -4.44479261962489E-05 1.56829556254391 -> xyz=0.0683718588662071 -0.00017216266999398 0.0965426886755783 rpy=1.26028779817361 -4.44479261962489E-05 1.56829556254391
- joint kinect_joint: origin xyz=-0.18135928471055 -0.175617930661629 0.749299999999995 rpy=3.14159265358979 -6.12296751932149E-17 -1.56621524571027 -> xyz=-0.2028 -0.18952 0.52978 rpy=1.5662 1.5708 0
- joint shoulder_roll_joint: origin xyz=0.0245928594915512 -0.0662368610105018 0 rpy=1.5707963267949 -0.00266644576657517 0.355511126450564 -> xyz=0.0245928594751605 -0.0662368609534871 0 rpy=1.5707963267949 -0.00266644576657517 0.355511126450564
- joint upper_arm_tracker_joint: origin xyz=0.0683718268361238 -0.000182515415244555 0.0965426841436375 rpy=1.26028781893805 -2.27414330644165E-05 1.56813717848772 -> xyz=0.0683718268246616 -0.000182516337945637 0.096542684260402 rpy=1.26028781893805 -2.27414330644165E-05 1.56813717848772
- joint wrist_lift_joint: origin xyz=-0.0114299633743926 2.87465063520953E-05 0.181015691120791 rpy=-1.5707963267949 -0.110406053363127 -0.00251502707069052 -> xyz=-0.0114299638504637 2.87467290271959E-05 0.181015691664385 rpy=-1.5707963267949 -0.110406053363127 -0.00251502707069052

Commit message: posture control working on old urdf

File: koko_descriptions/koko_description_sevendof_kin/robots/koko_description_sevendof_kin.urdf (robot description, URDF)
Before this commit: robot koko_description_sevendof_kin, 13 links, 12 joints
Joints:
- joint base_tracker_joint: origin xyz=0.122544343576621 0.0211413433675803 0.104502933199187 rpy=-0.00215895279379528 -0.78539656263699 -3.1385396042896 -> xyz=0.10380172 0.0211413433675803 0.13964323 rpy=-0.00215895279379528 -0.78539656263699 -3.1385396042896

Commit message: new URDF and current control code

File: koko_descriptions/koko_description_sevendof_kin/robots/koko_description_sevendof_kin.urdf (robot description, URDF)
Before this commit: robot koko_description_sevendof_kin, 13 links, 12 joints
Links:
- removed link kinet_link
- added link catcher_link, mass 0.210387685533954; collision mesh filename=package://koko_description_sevendof_kin/meshes/catcher_link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; visual mesh filename=package://koko_description_sevendof_kin/meshes/catcher_link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
- added link kinect_link, mass 0.141022435513688; collision mesh filename=package://koko_description_sevendof_kin/meshes/kinect_link.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; visual mesh filename=package://koko_description_sevendof_kin/meshes/kinect_link.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
- link forearm_link: mass 1.74772059521985 -> 1.74772059406253
- link forearm_tracker_link: mass 0.085205801529096 -> 0.0852058013520833
- link shoulder_lift_link: mass 0.491671117165989 -> 0.491670750547076
- link shoulder_link: mass 2.01456804587825 -> 2.01422165272683
- link upper_arm_lift_link: mass 0.4910945909981 -> 0.49109459100815
- link upper_arm_link: mass 1.74743726474448 -> 1.7476491152195
- link upper_arm_tracker_link: mass 0.0852060439090128 -> 0.0852060436498746
- link wrist_lift_link: mass 0.491088159923728 -> 0.491088159416964
- link wrist_link: mass 0.196389998403157 -> 0.196389984697673
Joints:
- added joint catcher_joint: type fixed, parent wrist_link, child catcher_link, origin xyz=0 0.11096 -0.0318679796126602 rpy=1.5707963267949 -1.5707963267949 -3.14159265358979, axis 0 0 0
- joint base_roll_joint: origin xyz=0.0901789447182363 -0.0908049999999997 0.212155832960628 rpy=6.83851519316138E-15 0.785398163397447 4.83556046633164E-15 -> xyz=0.090179 -0.090805 0.21216 rpy=6.8385E-15 0.7854 4.8356E-15
- joint base_tracker_joint: origin xyz=0.10380172 0.0211413433675803 0.13964323 rpy=-0.00215895279379528 -0.78539656263699 -3.1385396042896 -> xyz=0.035399 -0.090805 0.24718 rpy=-0.7854 6.123E-17 1.5708
- joint elbow_lift_joint: origin xyz=-0.0114299541998245 3.04774259364815E-05 0.181015677385081 rpy=-1.5707963267949 -0.355504877844586 -0.0026664457665753 -> xyz=-0.01143 3.0477E-05 0.18102 rpy=-1.5708 -0.3555 -0.0026664
- joint elbow_roll_joint: origin xyz=0.00778446382641085 -0.0702248716034493 0 rpy=1.5707963267949 -0.00251502707069075 0.11039980475715 -> xyz=0.0077845 -0.070225 0 rpy=1.5708 -0.002515 0.1104
- joint forearm_tracker_joint: origin xyz=0.0683718588661483 -0.000172162669981935 0.0965426886750276 rpy=1.26028779817361 -4.44479261962489E-05 1.56829556254391 -> xyz=0.068372 -0.00017216 0.096543 rpy=1.2603 -4.4448E-05 1.5683
- joint kinect_joint: child kinet_link -> kinect_link; origin xyz=0.0296663032719453 0.0534280083246514 0.655319999999998 rpy=-1.5707963267949 -1.5707963267949 -1.5707963267949 -> xyz=0.0296663032719453 0.0534280083246517 0.680719999999998 rpy=-1.5707963267949 -1.5707963267949 -1.5707963267949
- joint shoulder_lift_joint: origin xyz=0.0114299285786579 4.04065193964076E-05 0.210820000000001 rpy=1.5707963267949 -0.785395039094458 0.0035351359132397 -> xyz=0.01143 4.0407E-05 0.21082 rpy=1.5708 -0.7854 0.0035351
- joint shoulder_roll_joint: origin xyz=0.0245928619569141 -0.0662368676461337 0 rpy=1.5707963267949 -0.00266644576657517 0.355511126450564 -> xyz=0.024593 -0.066237 0 rpy=1.5708 -0.0026664 0.35551
- joint upper_arm_tracker_joint: origin xyz=0.0304107988383049 -7.9845769743736E-05 0.0425940035066137 rpy=1.26028781893822 -2.27414330359861E-05 1.56813717848771 -> xyz=0.0673059857243459 -0.000179630611320147 0.0961996133169819 rpy=1.26028690822204 0.00238258736259419 1.56736533514145
- joint wrist_lift_joint: origin xyz=-0.0114299638505801 2.87467290523424E-05 0.181015691663285 rpy=-1.5707963267949 -0.110406053363127 -0.00251502707069052 -> xyz=-0.0114299638605432 2.8746733649887E-05 0.181015691664515 rpy=-1.5707963267949 -0.110406053363127 -0.00251502707069052

Commit message: update from robot-reality-1

File: koko_descriptions/koko_description_sevendof_kin/robots/koko_description_sevendof_kin.urdf (robot description, URDF)
Before this commit: robot koko_description_sevendof_kin, 13 links, 12 joints
Links:
- removed link kinet_link
- added link catcher_link, mass 0.210387685533954; collision mesh filename=package://koko_description_sevendof_kin/meshes/catcher_link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; visual mesh filename=package://koko_description_sevendof_kin/meshes/catcher_link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
- added link kinect_link, mass 0.141022435513688; collision mesh filename=package://koko_description_sevendof_kin/meshes/kinect_link.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; visual mesh filename=package://koko_description_sevendof_kin/meshes/kinect_link.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
- link forearm_link: mass 1.74772059521985 -> 1.74772059406253
- link forearm_tracker_link: mass 0.085205801529096 -> 0.0852058013520833
- link shoulder_lift_link: mass 0.491671117165989 -> 0.491670750547076
- link shoulder_link: mass 2.01456804587825 -> 2.01422165272683
- link upper_arm_lift_link: mass 0.4910945909981 -> 0.49109459100815
- link upper_arm_link: mass 1.74743726474448 -> 1.7476491152195
- link upper_arm_tracker_link: mass 0.0852060439090128 -> 0.0852060436498746
- link wrist_lift_link: mass 0.491088159923728 -> 0.491088159416964
- link wrist_link: mass 0.196389998403157 -> 0.196389984697673
Joints:
- added joint catcher_joint: type fixed, parent wrist_link, child catcher_link, origin xyz=0 0.11096 -0.0318679796126602 rpy=1.5707963267949 -1.5707963267949 -3.14159265358979, axis 0 0 0
- joint base_roll_joint: origin xyz=0.0901789447182363 -0.0908049999999997 0.212155832960628 rpy=6.83851519316138E-15 0.785398163397447 4.83556046633164E-15 -> xyz=0.090179 -0.090805 0.21216 rpy=6.8385E-15 0.7854 4.8356E-15
- joint base_tracker_joint: origin xyz=0.104741193173153 0.0217020515197849 0.138021531898148 rpy=-0.00215895279379528 -0.78539656263699 -3.1385396042896 -> xyz=0.035399 -0.090805 0.24718 rpy=-0.7854 6.123E-17 1.5708
- joint elbow_lift_joint: origin xyz=-0.0114299541998245 3.04774259364815E-05 0.181015677385081 rpy=-1.5707963267949 -0.355504877844586 -0.0026664457665753 -> xyz=-0.01143 3.0477E-05 0.18102 rpy=-1.5708 -0.3555 -0.0026664
- joint elbow_roll_joint: origin xyz=0.00778446382641085 -0.0702248716034493 0 rpy=1.5707963267949 -0.00251502707069075 0.11039980475715 -> xyz=0.0077845 -0.070225 0 rpy=1.5708 -0.002515 0.1104
- joint forearm_tracker_joint: origin xyz=0.0683718588661483 -0.000172162669981935 0.0965426886750276 rpy=1.26028779817361 -4.44479261962489E-05 1.56829556254391 -> xyz=0.068372 -0.00017216 0.096543 rpy=1.2603 -4.4448E-05 1.5683
- joint kinect_joint: child kinet_link -> kinect_link; origin xyz=0.0296663032719453 0.0534280083246514 0.655319999999998 rpy=-1.5707963267949 -1.5707963267949 -1.5707963267949 -> xyz=0.0296663032719453 0.0534280083246517 0.680719999999998 rpy=-1.5707963267949 -1.5707963267949 -1.5707963267949
- joint shoulder_lift_joint: origin xyz=0.0114299285786579 4.04065193964076E-05 0.210820000000001 rpy=1.5707963267949 -0.785395039094458 0.0035351359132397 -> xyz=0.01143 4.0407E-05 0.21082 rpy=1.5708 -0.7854 0.0035351
- joint shoulder_roll_joint: origin xyz=0.0245928619569141 -0.0662368676461337 0 rpy=1.5707963267949 -0.00266644576657517 0.355511126450564 -> xyz=0.024593 -0.066237 0 rpy=1.5708 -0.0026664 0.35551
- joint upper_arm_tracker_joint: origin xyz=0.0304107988383049 -7.9845769743736E-05 0.0425940035066137 rpy=1.26028781893822 -2.27414330359861E-05 1.56813717848771 -> xyz=0.0673059857243459 -0.000179630611320147 0.0961996133169819 rpy=1.26028690822204 0.00238258736259419 1.56736533514145
- joint wrist_lift_joint: origin xyz=-0.0114299638505801 2.87467290523424E-05 0.181015691663285 rpy=-1.5707963267949 -0.110406053363127 -0.00251502707069052 -> xyz=-0.0114299638605432 2.8746733649887E-05 0.181015691664515 rpy=-1.5707963267949 -0.110406053363127 -0.00251502707069052
