Commit message: calibration changes & separated hw interface

File: koko_descriptions/koko_description_link/robots/koko_description_link.urdf (robot description, URDF)
Before this commit: robot koko_description_link, 3 links, 2 joints
Joints:
- joint lift_joint: limit lower=-2.2944 upper=0 effort=0 velocity=0 -> lower=-2.2944 upper=1.0 effort=0 velocity=0
