Commit message: New URDF

File: koko_descriptions/koko_description_sevendof_dyn/robots/koko_description_sevendof_dyn.urdf (robot description, URDF)
Before this commit: robot koko_description_sevendof_dyn, 8 links, 7 joints
Links:
- link base_link: mass 3.09843836934056 -> 5.30617493719281
- link forearm_link: mass 4.20066987914357 -> 1.83280962903355
- link shoulder_lift_link: mass 0.437261742773662 -> 0.491671117187525
- link shoulder_link: mass 4.07265346744175 -> 2.01456842992022
- link upper_arm_lift_link: mass 0.424523133438755 -> 0.491094590998026
- link upper_arm_link: mass 4.2742818546012 -> 1.83297890764661
- link wrist_lift_link: mass 0.475481880133678 -> 0.491088159417007
- link wrist_link: mass 1.09941045728339 -> 0.28159829590899
Joints:
- joint base_roll_joint: origin xyz=0.096645 -0.090805 0.21862 rpy=6.8385E-15 0.7854 4.8356E-15 -> xyz=0.0901789447182363 -0.0908049999999997 0.212155832960628 rpy=6.83851519316138E-15 0.785398163397447 4.83556046633164E-15
- joint elbow_lift_joint: origin xyz=-0.01143 3.0477E-05 0.18102 rpy=-1.5708 -0.3555 -0.0026664 -> xyz=-0.011429954204372 3.04766769116949E-05 0.181015691885107 rpy=-1.5707963267949 -0.355504877844586 -0.0026664457665753
- joint elbow_roll_joint: origin xyz=0.00778446382637513 -0.0702248716030744 0 rpy=1.5707963267949 -0.00251502707069075 0.11039980475715 -> xyz=0.00778446397719376 -0.070224872016303 0 rpy=1.5707963267949 -0.00251502707069075 0.11039980475715
- joint shoulder_lift_joint: origin xyz=0.01143 4.0407E-05 0.20168 rpy=1.5708 -0.7854 0.0035351 -> xyz=0.0114299285786579 4.04065193964076E-05 0.210820000000001 rpy=1.5707963267949 -0.785395039094458 0.0035351359132397
- joint shoulder_roll_joint: origin xyz=0.0245928594297677 -0.0662368608395588 0 rpy=1.5707963267949 -0.00266644576657517 0.355511126450564 -> xyz=0.0245928594422891 -0.0662368608700259 0 rpy=1.5707963267949 -0.00266644576657517 0.355511126450564
- joint wrist_joint: axis 0 0 -1 -> 0 -1 0; origin xyz=-0.0363404635750081 -0.0672158171493859 0 rpy=1.57079632679489 -0.00284167609972037 -0.49563904972794 -> xyz=-0.0115762893061741 -0.0214116626131124 0 rpy=1.62543589699027E-15 -1.18308141061618E-15 2.64595360386185
- joint wrist_lift_joint: origin xyz=-0.0114299638279672 2.87470080898022E-05 0.181015691624091 rpy=-1.5707963267949 -0.110406053363127 -0.00251502707069052 -> xyz=-0.011429964001298 2.8746722190276E-05 0.181015690796442 rpy=-1.5707963267949 -0.110406053363127 -0.00251502707069052

File: koko_descriptions/koko_description_sevendof_kin/robots/koko_description_sevendof_kin.urdf (robot description, URDF)
Before this commit: robot koko_description_sevendof_kin, 13 links, 12 joints
Links:
- removed link kinect_link
- added link kinet_link, mass 0.807440668573839; collision mesh filename=package://koko_description_sevendof_kin/meshes/kinet_link.S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; visual mesh filename=package://koko_description_sevendof_kin/meshes/kinet_link.S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
- link base_link: mass 3.09843836934056 -> 5.30617493719281
- link base_tracker_link: mass 0.0852031301907352 -> 0.0852057940282606
- link forearm_link: mass 4.11546002232608 -> 1.74772059521985
- link forearm_tracker_link: mass 0.0852058022688607 -> 0.085205801529096
- link shoulder_lift_link: mass 0.437261383344117 -> 0.491671117165989
- link shoulder_link: mass 4.07268991609326 -> 2.01456804587825
- link upper_arm_lift_link: mass 0.424523133438859 -> 0.4910945909981
- link upper_arm_link: mass 4.18907578737678 -> 1.74743726474448
- link upper_arm_tracker_link: mass 0.0852060551384698 -> 0.0852060439090128
- link wrist_lift_link: mass 0.475481880133676 -> 0.491088159923728
- link wrist_link: mass 1.01420215185203 -> 0.196389998403157
Joints:
- joint base_roll_joint: origin xyz=0.0966447291250239 -0.0908049999999999 0.218621617367798 rpy=6.83851519316138E-15 0.785398163397447 4.83556046633164E-15 -> xyz=0.0901789447182363 -0.0908049999999997 0.212155832960628 rpy=6.83851519316138E-15 0.785398163397447 4.83556046633164E-15
- joint base_tracker_joint: origin xyz=0.122544343576621 0.0211413433675803 0.104502933199187 rpy=-0.00215895279379528 -0.78539656263699 -3.1385396042896 -> xyz=0.104741193173153 0.0217020515197849 0.138021531898148 rpy=-0.00215895279379528 -0.78539656263699 -3.1385396042896
- joint ee_tracker_joint: origin xyz=0.000165588595298471 0.0582694656497648 0.0275400008691862 rpy=1.5707963267949 -3.52354834015197E-05 3.13875097749008 -> xyz=0 0.0796100008691862 0.058269700931892 rpy=1.09287578986539E-15 4.52676091056148E-15 3.52354834016303E-05
- joint elbow_lift_joint: origin xyz=-0.0114299548892374 3.04756154084207E-05 0.181015691851649 rpy=-1.5707963267949 -0.355504877844586 -0.0026664457665753 -> xyz=-0.0114299541998245 3.04774259364815E-05 0.181015677385081 rpy=-1.5707963267949 -0.355504877844586 -0.0026664457665753
- joint elbow_roll_joint: origin xyz=0.00778446477696024 -0.0702248702858572 0 rpy=1.5707963267949 -0.00251502707069075 0.11039980475715 -> xyz=0.00778446382641085 -0.0702248716034493 0 rpy=1.5707963267949 -0.00251502707069075 0.11039980475715
- joint forearm_tracker_joint: origin xyz=0.0683718588662071 -0.00017216266999398 0.0965426886755783 rpy=1.26028779817361 -4.44479261962489E-05 1.56829556254391 -> xyz=0.0683718588661483 -0.000172162669981935 0.0965426886750276 rpy=1.26028779817361 -4.44479261962489E-05 1.56829556254391
- joint kinect_joint: child kinect_link -> kinet_link; origin xyz=-0.2028 -0.18952 0.52978 rpy=1.5662 1.5708 0 -> xyz=0.0296663032719453 0.0534280083246514 0.655319999999998 rpy=-1.5707963267949 -1.5707963267949 -1.5707963267949
- joint shoulder_lift_joint: origin xyz=0.0114299285786579 4.04065193964076E-05 0.201676000000001 rpy=1.5707963267949 -0.785395039094458 0.0035351359132397 -> xyz=0.0114299285786579 4.04065193964076E-05 0.210820000000001 rpy=1.5707963267949 -0.785395039094458 0.0035351359132397
- joint shoulder_roll_joint: origin xyz=0.0245928594751605 -0.0662368609534871 0 rpy=1.5707963267949 -0.00266644576657517 0.355511126450564 -> xyz=0.0245928619569141 -0.0662368676461337 0 rpy=1.5707963267949 -0.00266644576657517 0.355511126450564
- joint upper_arm_tracker_joint: origin xyz=0.0683718268246616 -0.000182516337945637 0.096542684260402 rpy=1.26028781893805 -2.27414330644165E-05 1.56813717848772 -> xyz=0.0304107988383049 -7.9845769743736E-05 0.0425940035066137 rpy=1.26028781893822 -2.27414330359861E-05 1.56813717848771
- joint wrist_joint: axis 0 0 -1 -> 0 -1 0; origin xyz=-0.0363404635566231 -0.067215817115381 0 rpy=1.57079632679489 -0.00284167609972037 -0.49563904972794 -> xyz=-0.0115762892877892 -0.0214116625791075 0 rpy=1.62543589699027E-15 -1.18308141061618E-15 2.64595360386185
- joint wrist_lift_joint: origin xyz=-0.0114299638504637 2.87467290271959E-05 0.181015691664385 rpy=-1.5707963267949 -0.110406053363127 -0.00251502707069052 -> xyz=-0.0114299638505801 2.87467290523424E-05 0.181015691663285 rpy=-1.5707963267949 -0.110406053363127 -0.00251502707069052

Commit message: correct urdfs

File: koko_descriptions/koko_description_sevendof_dyn/robots/koko_description_sevendof_dyn.urdf (robot description, URDF)
Before this commit: robot koko_description_sevendof_dyn, 8 links, 7 joints
Links:
- removed link wrist_link
- added link wrist_roll_link, mass 1.49779120433657; collision mesh filename=package://koko_description_sevendof_dyn/meshes/wrist_roll_l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; visual mesh filename=package://koko_description_sevendof_dyn/meshes/wrist_roll_l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
- link base_link: mass 5.30617493719281 -> 0.210349130857436
- link forearm_link: mass 1.83280962903355 -> 4.12272375893646
- link shoulder_lift_link: mass 0.491671117187525 -> 0.437261741071288
- link shoulder_link: mass 2.01456842992022 -> 4.06056876982499
- link upper_arm_lift_link: mass 0.491094590998026 -> 0.437261171596556
- link upper_arm_link: mass 1.83297890764661 -> 4.20793381363064
- link wrist_lift_link: mass 0.491088159417007 -> 0.437254818113419
Joints:
- removed joint wrist_joint
- added joint wrist_roll_joint: type revolute, parent wrist_lift_link, child wrist_roll_link, origin xyz=-0.019428 -0.035935 0 rpy=-1.5708 -6.5009E-15 2.646, axis 0 0 -1, limit lower=-1.54 upper=1.54 effort=0 velocity=0
- joint base_roll_joint: limit (none) -> lower=-1.54 upper=1.54 effort=0 velocity=0; origin xyz=0.0901789447182363 -0.0908049999999997 0.212155832960628 rpy=6.83851519316138E-15 0.785398163397447 4.83556046633164E-15 -> xyz=0.011376 -0.15172 0.15127 rpy=6.8694E-15 0.7854 4.8574E-15; type continuous -> revolute
- joint elbow_lift_joint: axis 0 0 1 -> 1 0 0; limit (none) -> lower=-1.54 upper=1.54 effort=0 velocity=0; origin xyz=-0.011429954204372 3.04766769116949E-05 0.181015691885107 rpy=-1.5707963267949 -0.355504877844586 -0.0026664457665753 -> xyz=-0.011086 2.954E-05 0.18096 rpy=1.3274 -1.0278E-15 1.5681; type continuous -> revolute
- joint elbow_roll_joint: axis 0 0 -1 -> -1 0 0; limit (none) -> lower=-1.54 upper=1.54 effort=0 velocity=0; origin xyz=0.00778446397719376 -0.070224872016303 0 rpy=1.5707963267949 -0.00251502707069075 0.11039980475715 -> xyz=0 0.073871 0 rpy=-1.5708 1.6307E-15 1.5708; type continuous -> revolute
- joint shoulder_lift_joint: limit (none) -> lower=-1.54 upper=1.54 effort=0 velocity=0; origin xyz=0.0114299285786579 4.04065193964076E-05 0.210820000000001 rpy=1.5707963267949 -0.785395039094458 0.0035351359132397 -> xyz=0.01143 4.0407E-05 0.20168 rpy=1.5708 -0.7854 0.0035351; type continuous -> revolute
- joint shoulder_roll_joint: limit (none) -> lower=-1.54 upper=1.54 effort=0 velocity=0; origin xyz=0.0245928594422891 -0.0662368608700259 0 rpy=1.5707963267949 -0.00266644576657517 0.355511126450564 -> xyz=0.024591 -0.066323 0 rpy=1.5708 -0.0026647 0.35378; type continuous -> revolute
- joint wrist_lift_joint: limit (none) -> lower=-1.54 upper=1.54 effort=0 velocity=0; origin xyz=-0.011429964001298 2.8746722190276E-05 0.181015690796442 rpy=-1.5707963267949 -0.110406053363127 -0.00251502707069052 -> xyz=0.1778 0.01143 0 rpy=3.1416 -1.5135E-15 -1.4604; type continuous -> revolute

File: koko_descriptions/koko_description_sevendof_kin/robots/koko_description_sevendof_kin.urdf (robot description, URDF)
Before this commit: robot koko_description_sevendof_kin, 14 links, 13 joints
Links:
- removed link catcher_link
- removed link ee_tracker_link
- removed link kinect_link
- removed link wrist_link
- added link wrist_roll_link, mass 1.49779120356007; collision mesh filename=package://koko_description_sevendof_kin/meshes/wrist_roll_l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; visual mesh filename=package://koko_description_sevendof_kin/meshes/wrist_roll_l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
- link base_link: mass 5.30617493719281 -> 0.210349130781402
- link base_tracker_link: mass 0.0852057940282606 -> 0.0852058039730557
- link forearm_link: mass 1.74772059406253 -> 4.12272376366605
- link forearm_tracker_link: mass 0.0852058013520833 -> 0.0852058022688794
- link shoulder_lift_link: mass 0.491670750547076 -> 0.43726174275049
- link shoulder_link: mass 2.01422165272683 -> 4.06060300135281
- link upper_arm_lift_link: mass 0.49109459100815 -> 0.437261171586673
- link upper_arm_link: mass 1.7476491152195 -> 4.20793381703838
- link upper_arm_tracker_link: mass 0.0852060436498746 -> 0.0852060442329189
- link wrist_lift_link: mass 0.491088159416964 -> 0.437254818113419
Joints:
- removed joint catcher_joint
- removed joint ee_tracker_joint
- removed joint kinect_joint
- removed joint wrist_joint
- added joint wrist_roll_joint: type revolute, parent wrist_lift_link, child wrist_roll_link, origin xyz=-0.019428 -0.035935 0 rpy=-1.5708 -6.5009E-15 2.646, axis 0 0 -1, limit lower=-1.54 upper=1.54 effort=0 velocity=0
- joint base_roll_joint: limit (none) -> lower=-1.54 upper=1.54 effort=0 velocity=0; origin xyz=0.090179 -0.090805 0.21216 rpy=6.8385E-15 0.7854 4.8356E-15 -> xyz=0.011376 -0.15172 0.15127 rpy=6.8694E-15 0.7854 4.8574E-15; type continuous -> revolute
- joint base_tracker_joint: origin xyz=0.035399 -0.090805 0.24718 rpy=-0.7854 6.123E-17 1.5708 -> xyz=-0.0498692449226366 -0.151716256860219 0.179829435830465 rpy=-0.785398286004807 -5.15847808661681E-07 1.5707968426427
- joint elbow_lift_joint: axis 0 0 1 -> 1 0 0; limit (none) -> lower=-1.54 upper=1.54 effort=0 velocity=0; origin xyz=-0.01143 3.0477E-05 0.18102 rpy=-1.5708 -0.3555 -0.0026664 -> xyz=-0.01143 3.0476E-05 0.18102 rpy=1.3257 5.4262E-15 1.5681; type continuous -> revolute
- joint elbow_roll_joint: axis 0 0 -1 -> -1 0 0; limit (none) -> lower=-1.54 upper=1.54 effort=0 velocity=0; origin xyz=0.0077845 -0.070225 0 rpy=1.5708 -0.002515 0.1104 -> xyz=0 0.073871 0 rpy=-1.5708 1.6307E-15 1.5708; type continuous -> revolute
- joint forearm_tracker_joint: origin xyz=0.068372 -0.00017216 0.096543 rpy=1.2603 -4.4448E-05 1.5683 -> xyz=0.093326996938786 -0.0683720755168485 0 rpy=1.57079632696237 1.57074964653677 0.310508528471775
- joint shoulder_lift_joint: limit (none) -> lower=-1.54 upper=1.54 effort=0 velocity=0; origin xyz=0.01143 4.0407E-05 0.21082 rpy=1.5708 -0.7854 0.0035351 -> xyz=0.01143 4.0407E-05 0.20168 rpy=1.5708 -0.7854 0.0035351; type continuous -> revolute
- joint shoulder_roll_joint: limit (none) -> lower=-1.54 upper=1.54 effort=0 velocity=0; type continuous -> revolute
- joint upper_arm_tracker_joint: origin xyz=0.0673059857243459 -0.000179630611320147 0.0961996133169819 rpy=1.26028690822204 0.00238258736259419 1.56736533514145 -> xyz=0.0304107993735892 -7.98469833864779E-05 0.0425939383117631 rpy=1.26028779840761 -2.27414328887753E-05 1.56813717846785
- joint wrist_lift_joint: limit (none) -> lower=-1.54 upper=1.54 effort=0 velocity=0; origin xyz=-0.0114299638605432 2.8746733649887E-05 0.181015691664515 rpy=-1.5707963267949 -0.110406053363127 -0.00251502707069052 -> xyz=0.1778 0.01143 0 rpy=3.1416 -1.5135E-15 -1.4604; type continuous -> revolute

Commit message: Finalized and working new URDFs

File: koko_descriptions/koko_description_sevendof_dyn/robots/koko_description_sevendof_dyn.urdf (robot description, URDF)
Before this commit: robot koko_description_sevendof_dyn, 8 links, 7 joints
Joints:
- joint base_roll_joint: limit lower=-1.54 upper=1.54 effort=0 velocity=0 -> lower=-3 upper=3 effort=0 velocity=0
- joint elbow_lift_joint: limit lower=-1.54 upper=1.54 effort=0 velocity=0 -> lower=-3 upper=3 effort=0 velocity=0
- joint elbow_roll_joint: limit lower=-1.54 upper=1.54 effort=0 velocity=0 -> lower=-3 upper=3 effort=0 velocity=0
- joint shoulder_lift_joint: limit lower=-1.54 upper=1.54 effort=0 velocity=0 -> lower=-3 upper=3 effort=0 velocity=0
- joint shoulder_roll_joint: limit lower=-1.54 upper=1.54 effort=0 velocity=0 -> lower=-3 upper=3 effort=0 velocity=0
- joint wrist_lift_joint: limit lower=-1.54 upper=1.54 effort=0 velocity=0 -> lower=-3 upper=3 effort=0 velocity=0
- joint wrist_roll_joint: limit lower=-1.54 upper=1.54 effort=0 velocity=0 -> lower=-3 upper=3 effort=0 velocity=0

File: koko_descriptions/koko_description_sevendof_kin/robots/koko_description_sevendof_kin.urdf (robot description, URDF)
Before this commit: robot koko_description_sevendof_kin, 11 links, 10 joints
Links:
- added link ee_tracker_link, mass 0.0852083357798641; collision mesh filename=package://koko_description_sevendof_kin/meshes/ee_tracker_l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; visual mesh filename=package://koko_description_sevendof_kin/meshes/ee_tracker_l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
- link forearm_link: mass 4.12272376366605 -> 4.12272375225066
- link shoulder_lift_link: mass 0.43726174275049 -> 0.437261742750678
- link shoulder_link: mass 4.06060300135281 -> 4.06059384155066
- link upper_arm_lift_link: mass 0.437261171586673 -> 0.437261171596511
- link upper_arm_link: mass 4.20793381703838 -> 4.20794110984285
- link wrist_lift_link: mass 0.437254818113419 -> 0.437254818610311
- link wrist_roll_link: mass 1.49779120356007 -> 1.42202378562226
Joints:
- added joint ee_tracker_joint: type fixed, parent wrist_roll_link, child ee_tracker_link, origin xyz=0 -0.0465977473524162 0.0940905126607386 rpy=-1.5707963267949 3.52354834015197E-05 -3.14159265358978, axis 0 0 0
- joint base_roll_joint: limit lower=-1.54 upper=1.54 effort=0 velocity=0 -> lower=-3 upper=3 effort=0 velocity=0
- joint elbow_lift_joint: limit lower=-1.54 upper=1.54 effort=0 velocity=0 -> lower=-3 upper=3 effort=0 velocity=0
- joint elbow_roll_joint: limit lower=-1.54 upper=1.54 effort=0 velocity=0 -> lower=-3 upper=3 effort=0 velocity=0
- joint shoulder_lift_joint: limit lower=-1.54 upper=1.54 effort=0 velocity=0 -> lower=-3 upper=3 effort=0 velocity=0
- joint shoulder_roll_joint: limit lower=-1.54 upper=1.54 effort=0 velocity=0 -> lower=-3 upper=3 effort=0 velocity=0
- joint upper_arm_tracker_joint: origin xyz=0.0304107993735892 -7.98469833864779E-05 0.0425939383117631 rpy=1.26028779840761 -2.27414328887753E-05 1.56813717846785 -> xyz=0.068372 -0.00018252 0.096543 rpy=1.2603 -2.2741E-05 1.5681
- joint wrist_lift_joint: limit lower=-1.54 upper=1.54 effort=0 velocity=0 -> lower=-3 upper=3 effort=0 velocity=0
- joint wrist_roll_joint: limit lower=-1.54 upper=1.54 effort=0 velocity=0 -> lower=-3 upper=3 effort=0 velocity=0

Commit message: Created New URDF with specified conventions and exact soft joint limits

File: koko_descriptions/koko_description_sevendof_dyn/robots/koko_description_sevendof_dyn.urdf (robot description, URDF)
Before this commit: robot koko_description_sevendof_dyn, 8 links, 7 joints
Links:
- link base_link: mass 0.210349130857436 -> 1.94088320787417
- link forearm_link: mass 4.12272375893646 -> 1.60908907189915
- link shoulder_lift_link: mass 0.437261741071288 -> 0.388307110624732
- link shoulder_link: mass 4.06056876982499 -> 1.80875740468163
- link upper_arm_lift_link: mass 0.437261171596556 -> 0.336087766195346
- link upper_arm_link: mass 4.20793381363064 -> 1.60919074215694
- link wrist_lift_link: mass 0.437254818113419 -> 0.388307111938316
- link wrist_roll_link: mass 1.49779120433657 -> 0.332315567506482
Joints:
- joint base_roll_joint: limit lower=-3 upper=3 effort=0 velocity=0 -> lower=-2.3412 upper=3.3999 effort=0 velocity=0; origin xyz=0.011376 -0.15172 0.15127 rpy=6.8694E-15 0.7854 4.8574E-15 -> xyz=0.090179 -0.090805 0.21216 rpy=-3.1416 -0.7854 3.1416
- joint elbow_lift_joint: axis 1 0 0 -> 0 0 1; limit lower=-3 upper=3 effort=0 velocity=0 -> lower=-2.0944 upper=0 effort=0 velocity=0; origin xyz=-0.011086 2.954E-05 0.18096 rpy=1.3274 -1.0278E-15 1.5681 -> xyz=-0.01143 -4.0407E-05 -0.18056 rpy=-1.5708 -8.5189E-16 -3.1381
- joint elbow_roll_joint: axis -1 0 0 -> 0 0 1; limit lower=-3 upper=3 effort=0 velocity=0 -> lower=-2.6761 upper=2.6761 effort=0 velocity=0; origin xyz=0 0.073871 0 rpy=-1.5708 1.6307E-15 1.5708 -> xyz=0 0.070147 -6.25E-05 rpy=1.5708 -1.5708 0
- joint shoulder_lift_joint: limit lower=-3 upper=3 effort=0 velocity=0 -> lower=-2.0944 upper=0 effort=0 velocity=0; origin xyz=0.01143 4.0407E-05 0.20168 rpy=1.5708 -0.7854 0.0035351 -> xyz=-0.01143 0 -0.21082 rpy=-1.5708 4.4409E-16 3.1416
- joint shoulder_roll_joint: axis 0 0 -1 -> 0 0 1; limit lower=-3 upper=3 effort=0 velocity=0 -> lower=-2.6761 upper=2.6761 effort=0 velocity=0; origin xyz=0.024591 -0.066323 0 rpy=1.5708 -0.0026647 0.35378 -> xyz=0 0.070147 -6.25E-05 rpy=-1.5708 1.5673 -3.1416
- joint wrist_lift_joint: limit lower=-3 upper=3 effort=0 velocity=0 -> lower=-2.0944 upper=0 effort=0 velocity=0; origin xyz=0.1778 0.01143 0 rpy=3.1416 -1.5135E-15 -1.4604 -> xyz=-0.01143 0 -0.18056 rpy=-1.5708 6.6613E-16 -3.1416
- joint wrist_roll_joint: axis 0 0 -1 -> 0 0 1; limit lower=-3 upper=3 effort=0 velocity=0 -> lower=-2.6761 upper=2.6761 effort=0 velocity=0; origin xyz=-0.019428 -0.035935 0 rpy=-1.5708 -6.5009E-15 2.646 -> xyz=0 0.070147 -6.25E-05 rpy=-1.5708 -2.4803E-15 -3.1416

File: koko_descriptions/koko_description_sevendof_kin/robots/koko_description_sevendof_kin.urdf (robot description, URDF)
Before this commit: robot koko_description_sevendof_kin, 12 links, 11 joints
Links:
- link base_link: mass 0.210349130781402 -> 1.85567741361014
- link base_tracker_link: mass 0.0852058039730557 -> 0.0852057942640312
- link ee_tracker_link: mass 0.0852083357798641 -> 0.0852058039725329
- link forearm_link: mass 4.12272375225066 -> 1.52388327118307
- link forearm_tracker_link: mass 0.0852058022688794 -> 0.0852058007160938
- link shoulder_lift_link: mass 0.437261742750678 -> 0.388307110624734
- link shoulder_link: mass 4.06059384155066 -> 1.80875740468166
- link upper_arm_lift_link: mass 0.437261171596511 -> 0.336087766195304
- link upper_arm_link: mass 4.20794110984285 -> 1.52398195258296
- link upper_arm_tracker_link: mass 0.0852060442329189 -> 0.0852087895742651
- link wrist_lift_link: mass 0.437254818610311 -> 0.38830711159216
- link wrist_roll_link: mass 1.42202378562226 -> 0.247109756122906
Joints:
- joint base_roll_joint: limit lower=-3 upper=3 effort=0 velocity=0 -> lower=-2.3412 upper=3.3999 effort=0 velocity=0; origin xyz=0.011376 -0.15172 0.15127 rpy=6.8694E-15 0.7854 4.8574E-15 -> xyz=0.090179 -0.090805 0.21216 rpy=-3.1416 -0.7854 3.1416
- joint base_tracker_joint: origin xyz=-0.0498692449226366 -0.151716256860219 0.179829435830465 rpy=-0.785398286004807 -5.15847808661681E-07 1.5707968426427 -> xyz=0.034608 -0.090805 0.24797 rpy=-0.7854 1.4478E-14 1.5708
- joint ee_tracker_joint: origin xyz=0 -0.0465977473524162 0.0940905126607386 rpy=-1.5707963267949 3.52354834015197E-05 -3.14159265358978 -> xyz=0.046598 0 -0.063817 rpy=1.5708 -3.5235E-05 1.5708
- joint elbow_lift_joint: axis 1 0 0 -> 0 0 1; limit lower=-3 upper=3 effort=0 velocity=0 -> lower=-2.0944 upper=0 effort=0 velocity=0; origin xyz=-0.01143 3.0476E-05 0.18102 rpy=1.3257 5.4262E-15 1.5681 -> xyz=-0.01143 -4.0407E-05 -0.18056 rpy=-1.5708 -8.5189E-16 -3.1381
- joint elbow_roll_joint: axis -1 0 0 -> 0 0 1; limit lower=-3 upper=3 effort=0 velocity=0 -> lower=-2.6761 upper=2.6761 effort=0 velocity=0; origin xyz=0 0.073871 0 rpy=-1.5708 1.6307E-15 1.5708 -> xyz=0 0.070147 -6.25E-05 rpy=1.5708 -1.5708 0
- joint forearm_tracker_joint: origin xyz=0.093326996938786 -0.0683720755168485 0 rpy=1.57079632696237 1.57074964653677 0.310508528471775 -> xyz=0.068749 2.8791E-05 -0.096294 rpy=-1.8813 2.2741E-05 -1.5708
- joint shoulder_lift_joint: limit lower=-3 upper=3 effort=0 velocity=0 -> lower=-2.0944 upper=0 effort=0 velocity=0; origin xyz=0.01143 4.0407E-05 0.20168 rpy=1.5708 -0.7854 0.0035351 -> xyz=-0.01143 0 -0.21082 rpy=-1.5708 4.4409E-16 3.1416
- joint shoulder_roll_joint: axis 0 0 -1 -> 0 0 1; limit lower=-3 upper=3 effort=0 velocity=0 -> lower=-2.6761 upper=2.6761 effort=0 velocity=0; origin xyz=0.024593 -0.066237 0 rpy=1.5708 -0.0026664 0.35551 -> xyz=0 0.070147 -6.25E-05 rpy=-1.5708 1.5673 -3.1416
- joint upper_arm_tracker_joint: origin xyz=0.068372 -0.00018252 0.096543 rpy=1.2603 -2.2741E-05 1.5681 -> xyz=0.068748 0.00027183 -0.096294 rpy=-1.8813 2.2741E-05 -1.5673
- joint wrist_lift_joint: limit lower=-3 upper=3 effort=0 velocity=0 -> lower=-2.0944 upper=0 effort=0 velocity=0; origin xyz=0.1778 0.01143 0 rpy=3.1416 -1.5135E-15 -1.4604 -> xyz=-0.01143 0 -0.18056 rpy=-1.5708 6.6613E-16 -3.1416
- joint wrist_roll_joint: axis 0 0 -1 -> 0 0 1; limit lower=-3 upper=3 effort=0 velocity=0 -> lower=-2.6761 upper=2.6761 effort=0 velocity=0; origin xyz=-0.019428 -0.035935 0 rpy=-1.5708 -6.5009E-15 2.646 -> xyz=0 0.070147 -6.25E-05 rpy=-1.5708 -2.4803E-15 -3.1416
