Commit message: persistent calibration values

File: koko_descriptions/koko_description_sevendof_dyn/robots/koko_description_sevendof_dyn.urdf (robot description, URDF)
Before this commit: robot koko_description_sevendof_dyn, 8 links, 7 joints
Links:
- link wrist_roll_link: mass 0.802315567506482 -> 0.752315567506482

Commit message: updated urdf to be more general for using with accelerometers

File: koko_descriptions/koko_description_sevendof_dyn/robots/koko_description_sevendof_dyn.urdf (robot description, URDF)
Before this commit: robot koko_description_sevendof_dyn, 8 links, 7 joints
Links:
- link base_link: mass 1.94088320787417 -> 0.284612172465311
- link forearm_link: mass 1.60908907189915 -> 1.52367945216034
- link shoulder_lift_link: mass 0.488307110624732 -> 0.388307108622636
- link shoulder_link: mass 1.80875740468163 -> 1.80901122392276
- link upper_arm_lift_link: mass 0.488307110624732 -> 0.336087767400233
- link upper_arm_link: mass 1.80875740468163 -> 1.52396434922939
- link wrist_lift_link: mass 0.488307111938316 -> 0.388307111315058
- link wrist_roll_link: mass 0.752315567506482 -> 0.247109755986862
Joints:
- joint base_roll_joint: origin xyz=0.090179 -0.090805 0.21216 rpy=-3.1416 -0.7854 3.1416 -> xyz=0 0 0.054356 rpy=3.1416 -2.2011E-29 3.1416

File: koko_descriptions/koko_description_sevendof_kin/robots/koko_description_sevendof_kin.urdf (robot description, URDF)
Before this commit: robot koko_description_sevendof_kin, 12 links, 11 joints
Links:
- link base_link: mass 1.85567741361014 -> 0.284612172465311
- link base_tracker_link: mass 0.0852057942640312 -> 0.0852057942640298
- link ee_tracker_link: mass 0.0852058039725329 -> 0.0852058039712401
- link forearm_link: mass 1.52388327118307 -> 1.52407731945949
- link forearm_tracker_link: mass 0.0852058007160938 -> 0.0852058014578218
- link shoulder_lift_link: mass 0.388307110624734 -> 0.388307108622635
- link shoulder_link: mass 1.80875740468166 -> 1.80901122392277
- link upper_arm_lift_link: mass 0.336087766195304 -> 0.336087766639304
- link upper_arm_link: mass 1.52398195258296 -> 1.52396434922932
- link upper_arm_tracker_link: mass 0.0852087895742651 -> 0.0852087902897732
- link wrist_lift_link: mass 0.38830711159216 -> 0.388307109282073
- link wrist_roll_link: mass 0.247109756122906 -> 0.247109755986862
Joints:
- joint base_roll_joint: origin xyz=0.090179 -0.090805 0.21216 rpy=-3.1416 -0.7854 3.1416 -> xyz=0 0 0.054356 rpy=3.1416 -2.2011E-29 3.1416
- joint base_tracker_joint: origin xyz=0.034608 -0.090805 0.24797 rpy=-0.7854 1.4478E-14 1.5708 -> xyz=-0.0646197009318908 0 0.0403859991257779 rpy=-1.57079632679489 -3.56673679882293E-18 1.57079632679489
- joint forearm_tracker_joint: origin xyz=0.068749 2.8791E-05 -0.096294 rpy=-1.8813 2.2741E-05 -1.5708 -> xyz=0.0687486075198113 2.87912553707526E-05 -0.0962935677600952 rpy=-1.88130485518218 2.27414328835253E-05 -1.57080362425475
- joint upper_arm_tracker_joint: origin xyz=0.068748 0.00027183 -0.096294 rpy=-1.8813 2.2741E-05 -1.5673 -> xyz=0.0687480716074886 0.000271826226759544 -0.0962935663002703 rpy=-1.88130485518218 2.2741432881685E-05 -1.56726848834151

Commit message: Modular Hardware interface code! updated URDF to make more sense in current context of arm mounting

File: koko_descriptions/koko_description_sevendof_dyn/robots/koko_description_sevendof_dyn.urdf (robot description, URDF)
Before this commit: robot koko_description_sevendof_dyn, 8 links, 7 joints
Joints:
- joint base_roll_joint: origin xyz=0 0 0.054356 rpy=3.1416 -2.2011E-29 3.1416 -> xyz=0 0 0.054356 rpy=3.1416 -2.2011E-29 0.0

File: koko_descriptions/koko_description_sevendof_kin/robots/koko_description_sevendof_kin.urdf (robot description, URDF)
Before this commit: robot koko_description_sevendof_kin, 12 links, 11 joints
Joints:
- joint base_roll_joint: origin xyz=0 0 0.054356 rpy=3.1416 -2.2011E-29 3.1416 -> xyz=0 0 0.054356 rpy=3.1416 -2.2011E-29 0

Commit message: Gripper is integrated in control code!

File: koko_descriptions/koko_description_sevendof_dyn/robots/koko_description_sevendof_dyn.urdf (robot description, URDF)
Before this commit: robot koko_description_sevendof_dyn, 8 links, 7 joints
Links:
- added link gripper_link, mass 0.047109755986862; collision mesh filename=package://koko_description_sevendof_dyn/meshes/wrist_roll_l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; visual mesh filename=package://koko_description_sevendof_dyn/meshes/wrist_roll_l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
Joints:
- added joint gripper_joint: type revolute, parent wrist_roll_link, child gripper_link, origin xyz=0 0.070147 -6.25E-05 rpy=-1.5708 -2.4803E-15 -3.1416, axis 0 0 1, limit lower=-2.6761 upper=2.6761 effort=0 velocity=0

File: koko_descriptions/koko_description_sevendof_kin/robots/koko_description_sevendof_kin.urdf (robot description, URDF)
Before this commit: robot koko_description_sevendof_kin, 12 links, 11 joints
Links:
- added link gripper_link, mass 0.047109755986862; collision mesh filename=package://koko_description_sevendof_dyn/meshes/wrist_roll_l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; visual mesh filename=package://koko_description_sevendof_dyn/meshes/wrist_roll_l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
Joints:
- added joint gripper_joint: type revolute, parent wrist_roll_link, child gripper_link, origin xyz=0 0.070147 -6.25E-05 rpy=-1.5708 -2.4803E-15 -3.1416, axis 0 0 1, limit lower=-2.6761 upper=2.6761 effort=0 velocity=0

Commit message: koko_description is now a right arm

File: koko_descriptions/koko_description_sevendof_dyn/robots/koko_description_sevendof_dyn.urdf (robot description, URDF)
Before this commit: robot koko_description_sevendof_dyn, 9 links, 8 joints
Joints:
- joint base_roll_joint: limit lower=-2.3412 upper=3.3999 effort=0 velocity=0 -> lower=-3.3999 upper=2.3412 effort=0 velocity=0
- joint elbow_roll_joint: origin xyz=0 0.070147 -6.25E-05 rpy=1.5708 -1.5708 0 -> xyz=0 0.070147 -6.25E-05 rpy=1.5708 1.5708 0
- joint shoulder_roll_joint: origin xyz=0 0.070147 -6.25E-05 rpy=-1.5708 1.5673 -3.1416 -> xyz=0 0.070147 -6.25E-05 rpy=-1.5708 -1.5673 -3.1416

File: koko_descriptions/koko_description_sevendof_kin/robots/koko_description_sevendof_kin.urdf (robot description, URDF)
Before this commit: robot koko_description_sevendof_kin, 13 links, 12 joints
Joints:
- joint base_roll_joint: limit lower=-2.3412 upper=3.3999 effort=0 velocity=0 -> lower=-3.3999 upper=2.3412 effort=0 velocity=0
- joint elbow_roll_joint: origin xyz=0 0.070147 -6.25E-05 rpy=1.5708 -1.5708 0 -> xyz=0 0.070147 -6.25E-05 rpy=1.5708 1.5708 0
- joint shoulder_roll_joint: origin xyz=0 0.070147 -6.25E-05 rpy=-1.5708 1.5673 -3.1416 -> xyz=0 0.070147 -6.25E-05 rpy=-1.5708 -1.5673 -3.1416

Commit message: improved stability of CartesianPose Controller

File: koko_descriptions/koko_description_sevendof_dyn/robots/koko_description_sevendof_dyn.urdf (robot description, URDF)
Before this commit: robot koko_description_sevendof_dyn, 9 links, 8 joints
Links:
- link gripper_link: mass 0.047109755986862 -> 0.0047109755986862
- link shoulder_lift_link: mass 0.388307108622636 -> 0.488307108622636
- link shoulder_link: mass 1.80901122392276 -> 1.90901122392276
- link upper_arm_lift_link: mass 0.336087767400233 -> 0.436087767400233
- link upper_arm_link: mass 1.52396434922939 -> 1.92396434922939
- link wrist_lift_link: mass 0.388307111315058 -> 0.488307111315058
- link wrist_roll_link: mass 0.247109755986862 -> 0.657109755986862
Joints:
- joint wrist_roll_joint: origin xyz=0 0.070147 -6.25E-05 rpy=-1.5708 -2.4803E-15 -3.1416 -> xyz=0 0.170147 -6.25E-05 rpy=-1.5708 -2.4803E-15 -3.1416

File: koko_descriptions/koko_description_sevendof_kin/robots/koko_description_sevendof_kin.urdf (robot description, URDF)
Before this commit: robot koko_description_sevendof_kin, 13 links, 12 joints
Joints:
- joint wrist_roll_joint: origin xyz=0 0.070147 -6.25E-05 rpy=-1.5708 -2.4803E-15 -3.1416 -> xyz=0 0.170147 -6.25E-05 rpy=-1.5708 -2.4803E-15 -3.1416

Commit message: clean up and adjusted urdf masses

File: koko_descriptions/koko_description_sevendof_dyn/robots/koko_description_sevendof_dyn.urdf (robot description, URDF)
Before this commit: robot koko_description_sevendof_dyn, 9 links, 8 joints
Links:
- link forearm_link: mass 1.52367945216034 -> 1.42367945216034
