Commit message: finished xacros

File: koko_descriptions/koko_description_sevendof/robots/koko_arm.urdf.xacro (robot description, xacro)
@@ -6,4 +6,5 @@
   <xacro:include filename="$(find koko_description_sevendof)/urdf/base_v0/base.urdf.xacro" />
   <xacro:include filename="$(find koko_description_sevendof)/urdf/link_v0/link.urdf.xacro" />
+  <xacro:include filename="$(find koko_description_sevendof)/urdf/gripper_v0/gripper.urdf.xacro" />
   <!-- <xacro:include filename="$(find koko_description_sevendof)/urdf/upper_arm_v0/upper_arm.urdf.xacro" /> -->
   <!-- <xacro:include filename="$(find koko_description_sevendof)/urdf/forearm_v0/forearm.urdf.xacro" /> -->
@@ -20,5 +21,6 @@
   <xacro:koko_base_v0 side="right" reflect="-1" child="shoulder_roll_link"/>
   <xacro:koko_link_v0 side="right" stage="shoulder" child="upper_arm_roll_link" reflect="-1"/>
-  <xacro:koko_link_v0 side="right" stage="upper_arm" child="elbow_roll_link" reflect="-1"/>
-  <xacro:koko_link_v0 side="right" stage="elbow" child="wrist_roll_link" reflect="-1"/>
+  <xacro:koko_link_v0 side="right" stage="upper_arm" child="elbow_roll_link" reflect="1"/>
+  <xacro:koko_link_v0 side="right" stage="elbow" child="wrist_roll_link" reflect="0"/>
+  <xacro:koko_end_effector_v0 side="right" name="wrist_roll_link"/>
 </robot>

File: koko_descriptions/koko_description_sevendof/urdf/base_v0/base.urdf.xacro (robot description, xacro)
@@ -53,5 +53,5 @@
       type="revolute">
       <origin
-        xyz="0 0 0.054356"
+        xyz="0 0 0.087371"
         rpy="3.1416 -2.2011E-29 0.0" />
       <parent

File: koko_descriptions/koko_description_sevendof/urdf/gripper_v0/gripper.urdf.xacro (robot description, xacro)
@@ -23,11 +23,11 @@
   <!-- ============================  link  ============================ -->
   <!-- Includes elbow flex, FA roll joints in macros below -->
-  <xacro:macro name="koko_link_v0" params="side stage child reflect">
-    <xacro:koko_roll_link_v0 side="${side}" stage="${stage}" reflect="${reflect}" />
-    <xacro:koko_lift_link_v0 side="${side}" stage="${stage}" child="${child}" reflect="${reflect}" />
+  <xacro:macro name="koko_end_effector_v0" params="side name">
+    <xacro:koko_end_v0 side="${side}" name="${name}"/>
+    <xacro:koko_gripper_v0 side="${side}" parent="${name}"/>
   </xacro:macro>
-  <xacro:macro name="koko_roll_link_v0" params="side stage reflect">
+  <xacro:macro name="koko_end_v0" params="side name">
     <link
-      name="${side}_${stage}_roll_link">
+      name="${side}_${name}">
       <inertial>
         <origin
@@ -50,5 +50,5 @@
         <geometry>
           <mesh
-            filename="package://koko_description_sevendof/meshes/roll_link.STL" />
+            filename="package://koko_description_sevendof/meshes/wrist_roll_link.STL" />
         </geometry>
         <material
@@ -64,43 +64,25 @@
         <geometry>
           <mesh
-            filename="package://koko_description_sevendof/meshes/roll_link.STL" />
+            filename="package://koko_description_sevendof/meshes/wrist_roll_link.STL" />
         </geometry>
       </collision>
     </link>
-    <joint
-      name="${side}_${stage}_lift_joint"
-      type="revolute">
-      <origin
-        xyz="-0.01143 0 -0.18056"
-        rpy="-1.5708 4.4409E-16 3.1416" />
-      <parent
-        link="${side}_${stage}_roll_link"/>
-      <child
-        link="${side}_${stage}_lift_link"/>
-      <axis
-        xyz="0 0 1" />
-      <limit
-        lower="-2.2944"
-        upper="0"
-        effort="0"
-        velocity="0" />
-    </joint>
   </xacro:macro>
-  <xacro:macro name="koko_lift_link_v0" params="side stage child reflect">
+  <xacro:macro name="koko_gripper_v0" params="side parent">
     <link
-      name="${side}_${stage}_lift_link">
+      name="${side}_gripper_link">
       <inertial>
         <origin
-          xyz="-5.0083559080677E-06 0.000232928456050885 -1.77451392545103E-05"
+          xyz="-7.00549073506807E-05 2.51271935254316E-05 -0.052367118189184"
           rpy="0 0 0" />
         <mass
-          value="0.488307108622636" />
+          value="0.0047109755986862" />
         <inertia
-          ixx="0.000804272985961788"
-          ixy="4.84548777859872E-08"
-          ixz="2.09160815704306E-06"
-          iyy="0.000818260636171894"
-          iyz="-1.44954778549764E-08"
-          izz="0.000550840705045094" />
+          ixx="0.000916887873826385"
+          ixy="-6.04547948818479E-08"
+          ixz="0.6796133363069E-06"
+          iyy="0.000877268801166351"
+          iyz="0.64172907801915E-07"
+          izz="0.000293333065172452" />
       </inertial>
       <visual>
@@ -110,5 +92,5 @@
         <geometry>
           <mesh
-            filename="package://koko_description_sevendof/meshes/lift_link.STL" />
+            filename="package://koko_description_sevendof/meshes/wrist_roll_link.STL" />
         </geometry>
         <material
@@ -124,18 +106,18 @@
         <geometry>
           <mesh
-            filename="package://koko_description_sevendof/meshes/lift_link.STL" />
+            filename="package://koko_description_sevendof/meshes/wrist_roll_link.STL" />
         </geometry>
       </collision>
     </link>
     <joint
-      name="${side}_${stage}_roll_joint"
+      name="${side}_gripper_joint"
       type="revolute">
       <origin
         xyz="0 0.070147 -6.25E-05"
-        rpy="-1.5708 ${reflect*1.5673} -3.1416" />
+        rpy="-1.5708 -2.4803E-15 -3.1416" />
       <parent
-        link="${side}_${stage}_lift_link"/>
+        link="${side}_${parent}" />
       <child
-        link="${side}_${child}" />
+        link="${side}_gripper_link" />
       <axis
         xyz="0 0 1" />
