Commit message: added xacros support to launching arm

File: koko_descriptions/koko_description_sevendof/robots/koko_right_arm.urdf.xacro (robot description, xacro)
@@ -20,7 +20,7 @@
        is the world frame). For more, see http://www.ros.org/wiki/xacro -->
   <xacro:koko_base_v0 side="right" reflect="-1" child="shoulder_roll_link"/>
-  <xacro:koko_link_v0 side="right" stage="shoulder" child="upper_arm_roll_link" reflect="-1"/>
-  <xacro:koko_link_v0 side="right" stage="upper_arm" child="elbow_roll_link" reflect="1"/>
-  <xacro:koko_link_v0 side="right" stage="elbow" child="wrist_roll_link" reflect="0"/>
-  <xacro:koko_end_effector_v0 side="right" name="wrist_roll_link"/>
+  <xacro:koko_link_v0 side="right" stage="shoulder" child="elbow_roll_link" reflect="-1" />
+  <xacro:koko_link_v0 side="right" stage="elbow" child="wrist_roll_link" reflect="1" />
+  <xacro:koko_link_v0 side="right" stage="wrist" child="end_roll_link" reflect="0" wrist="1"/>
+  <xacro:koko_end_effector_v0 side="right" name="end_roll_link"/>
 </robot>

File: koko_descriptions/koko_description_sevendof/urdf/gripper_v0/gripper.urdf.xacro (robot description, xacro)
@@ -35,5 +35,5 @@
           rpy="0 0 0" />
         <mass
-          value="1.92367945216034" />
+          value="0.657109755986862" />
         <inertia
           ixx="0.0057866591250737"

File: koko_descriptions/koko_description_sevendof/urdf/link_v0/link.urdf.xacro (robot description, xacro)
@@ -23,9 +23,9 @@
   <!-- ============================  link  ============================ -->
   <!-- Includes elbow flex, FA roll joints in macros below -->
-  <xacro:macro name="koko_link_v0" params="side stage child reflect">
-    <xacro:koko_roll_link_v0 side="${side}" stage="${stage}" reflect="${reflect}" />
+  <xacro:macro name="koko_link_v0" params="side stage child reflect wrist:=0">
+    <xacro:koko_roll_link_v0 side="${side}" stage="${stage}" reflect="${reflect}" wrist="${wrist}"/>
     <xacro:koko_lift_link_v0 side="${side}" stage="${stage}" child="${child}" reflect="${reflect}" />
   </xacro:macro>
-  <xacro:macro name="koko_roll_link_v0" params="side stage reflect">
+  <xacro:macro name="koko_roll_link_v0" params="side stage reflect wrist">
     <link
       name="${side}_${stage}_roll_link">
@@ -35,5 +35,5 @@
           rpy="0 0 0" />
         <mass
-          value="1.92367945216034" />
+          value="${1.91396434922939 - 0.50028 * wrist}" />
         <inertia
           ixx="0.0057866591250737"
@@ -95,5 +95,5 @@
           rpy="0 0 0" />
         <mass
-          value="0.488307108622636" />
+          value="0.448307108622636" />
         <inertia
           ixx="0.000804272985961788"
