Commit message: added transmissions and gazebo parameter

File: blue_descriptions/robots/blue_left.urdf.xacro (robot description, xacro)
@@ -1,4 +1,6 @@
 <?xml version="1.0"?>
 <robot xmlns:xacro="http://ros.org/wiki/xacro" name="blue_descriptions_right">
+  <xacro:arg name="is_gazebo" default="false" />
+  <xacro:property name="is_gazebo" value="$(arg is_gazebo)" />
   <xacro:include filename="$(find blue_descriptions)/urdf/base_v0/base.urdf.xacro" />
   <xacro:include filename="$(find blue_descriptions)/urdf/link_v0/link.urdf.xacro" />

File: blue_descriptions/robots/blue_right.urdf.xacro (robot description, xacro)
@@ -1,4 +1,6 @@
 <?xml version="1.0"?>
 <robot xmlns:xacro="http://ros.org/wiki/xacro" name="blue_descriptions_right">
+  <xacro:arg name="is_gazebo" default="false" />
+  <xacro:property name="is_gazebo" value="$(arg is_gazebo)" />
   <xacro:include filename="$(find blue_descriptions)/urdf/base_v0/base.urdf.xacro" />
   <xacro:include filename="$(find blue_descriptions)/urdf/link_v0/link.urdf.xacro" />

File: blue_descriptions/urdf/base_v0/base.urdf.xacro (robot description, xacro)
@@ -73,5 +73,5 @@
           <hardwareInterface>EffortJointInterface</hardwareInterface>
         </joint>
-        <actuator name="{side}_base_roll_motor">
+        <actuator name="${side}_base_roll_motor">
           <hardwareInterface>EffortJointInterface</hardwareInterface>
           <mechanicalReduction>1</mechanicalReduction>

File: blue_descriptions/urdf/gripper_v0/gripper.urdf.xacro (robot description, xacro)
@@ -108,4 +108,16 @@
         velocity="0" />
     </joint>
+    <xacro:if value="${is_gazebo}">
+      <transmission name="${side}_gripper_transmission">
+        <type>transmission_interface/SimpleTransmission</type>
+        <joint name="${side}_gripper_joint">
+          <hardwareInterface>EffortJointInterface</hardwareInterface>
+        </joint>
+        <actuator name="${side}_gripper_motor">
+          <hardwareInterface>EffortJointInterface</hardwareInterface>
+          <mechanicalReduction>1</mechanicalReduction>
+        </actuator>
+      </transmission>
+    </xacro:if>
   </xacro:macro>
 </robot>

File: blue_descriptions/urdf/link_v0/link.urdf.xacro (robot description, xacro)
@@ -67,4 +67,16 @@
         velocity="0" />
     </joint>
+    <xacro:if value="${is_gazebo}">
+      <transmission name="${side}_${stage}_lift_joint_transmission">
+        <type>transmission_interface/SimpleTransmission</type>
+        <joint name="${side}_${stage}_lift_joint">
+          <hardwareInterface>EffortJointInterface</hardwareInterface>
+        </joint>
+        <actuator name="${side}_${stage}_lift_motor">
+          <hardwareInterface>EffortJointInterface</hardwareInterface>
+          <mechanicalReduction>1</mechanicalReduction>
+        </actuator>
+      </transmission>
+    </xacro:if>
   </xacro:macro>
   <xacro:macro name="blue_lift_link_v0" params="side stage child reflect">
@@ -127,4 +139,16 @@
         velocity="0" />
     </joint>
+    <xacro:if value="${is_gazebo}">
+      <transmission name="${side}_${stage}_roll_joint_transmission">
+        <type>transmission_interface/SimpleTransmission</type>
+        <joint name="${side}_${stage}_roll_joint">
+          <hardwareInterface>EffortJointInterface</hardwareInterface>
+        </joint>
+        <actuator name="${side}_${stage}_roll_motor">
+          <hardwareInterface>EffortJointInterface</hardwareInterface>
+          <mechanicalReduction>1</mechanicalReduction>
+        </actuator>
+      </transmission>
+    </xacro:if>
   </xacro:macro>
 </robot>
