Commit message: working blue in gazbo, need to add transmissions

File: blue_descriptions/robots/blue_full.urdf.xacro (robot description, xacro)
@@ -1,18 +1,15 @@
 <?xml version="1.0"?>
 <robot xmlns:xacro="http://ros.org/wiki/xacro" name="blue_descriptions_right">
-  <xacro:include filename="$(find blue_descriptions)/urdf/base_v0/base.urdf.xacro" />
-  <xacro:include filename="$(find blue_descriptions)/urdf/link_v0/link.urdf.xacro" />
-  <xacro:include filename="$(find blue_descriptions)/urdf/gripper_v0/gripper.urdf.xacro" />
+  <xacro:arg name="is_gazebo" default="false" />
+  <xacro:property name="is_gazebo" value="$(arg is_gazebo)" />
+  <!-- ====== Load in robot base macro ====== -->
   <xacro:include filename="$(find blue_descriptions)/urdf/robot_base_v0/robot_base.urdf.xacro" />
-  <xacro:blue_robot_base_v0 />
-  <xacro:blue_base_v0 side="right" reflect="-1" child="shoulder_roll_link"/>
-  <xacro:blue_link_v0 side="right" stage="shoulder" child="elbow_roll_link" reflect="-1" />
-  <xacro:blue_link_v0 side="right" stage="elbow" child="wrist_roll_link" reflect="1" />
-  <xacro:blue_link_v0 side="right" stage="wrist" child="end_roll_link" reflect="0" wrist="1"/>
-  <xacro:blue_end_effector_v0 side="right" name="end_roll_link"/>
-  <xacro:blue_base_v0 side="left" reflect="1" child="shoulder_roll_link"/>
-  <xacro:blue_link_v0 side="left" stage="shoulder" child="elbow_roll_link" reflect="1" />
-  <xacro:blue_link_v0 side="left" stage="elbow" child="wrist_roll_link" reflect="-1" />
-  <xacro:blue_link_v0 side="left" stage="wrist" child="end_roll_link" reflect="0" wrist="1"/>
-  <xacro:blue_end_effector_v0 side="left" name="end_roll_link"/>
+  <!-- ====== Robot camera height and angle parameters  ====== -->
+  <xacro:property name="base_camera_height"  value="0.303506965011826" />
+  <xacro:property name="camera_angle"  value= "0.0" />
+  <!-- ====== Build base ====== -->
+  <xacro:blue_robot_base_v0 cam_height="${base_camera_height}" cam_angle="${camera_angle}" is_gazebo="${is_gazebo}"/>
+  <!-- ====== Build right and left arms====== -->
+  <xacro:include filename="$(find blue_descriptions)/robots/blue_right.urdf.xacro" />
+  <xacro:include filename="$(find blue_descriptions)/robots/blue_left.urdf.xacro" />
 </robot>

File: blue_descriptions/robots/blue_right.urdf.xacro (robot description, xacro)
@@ -1,22 +1,7 @@
 <?xml version="1.0"?>
 <robot xmlns:xacro="http://ros.org/wiki/xacro" name="blue_descriptions_right">
-  <!-- The following included files set up definitions of parts of the robot body -->
-  <!-- misc common stuff? -->
-  <!-- PR2 Arm -->
   <xacro:include filename="$(find blue_descriptions)/urdf/base_v0/base.urdf.xacro" />
   <xacro:include filename="$(find blue_descriptions)/urdf/link_v0/link.urdf.xacro" />
   <xacro:include filename="$(find blue_descriptions)/urdf/gripper_v0/gripper.urdf.xacro" />
-  <!-- <xacro:include filename="$(find blue_descriptions)/urdf/upper_arm_v0/upper_arm.urdf.xacro" /> -->
-  <!-- <xacro:include filename="$(find blue_descriptions)/urdf/forearm_v0/forearm.urdf.xacro" /> -->
-  <!-- PR2 gripper -->
-  <!-- <xacro:include filename="$(find pr2_description)/urdf/gripper_v0/gripper.urdf.xacro" /> -->
-  <!-- Now we can start using the macros included above to define the actual PR2 -->
-  <!-- The first use of a macro.  This one was defined in base.urdf.xacro above.
-       A macro like this will expand to a set of link and joint definitions, and to additional
-       Gazebo-related extensions (sensor plugins, etc).  The macro takes an argument, name,
-       that equals "base", and uses it to generate names for its component links and joints
-       (e.g., base_link).  The included origin block is also an argument to the macro.  By convention,
-       the origin block defines where the component is w.r.t its parent (in this case the parent
-       is the world frame). For more, see http://www.ros.org/wiki/xacro -->
   <xacro:blue_base_v0 side="right" reflect="-1" child="shoulder_roll_link"/>
   <xacro:blue_link_v0 side="right" stage="shoulder" child="elbow_roll_link" reflect="-1" />

File: blue_descriptions/urdf/base_v0/base.urdf.xacro (robot description, xacro)
@@ -67,4 +67,16 @@
         velocity="0" />
     </joint>
+    <xacro:if value="${is_gazebo}">
+      <transmission name="${side}_base_roll_joint_transmission">
+        <type>transmission_interface/SimpleTransmission</type>
+        <joint name="${side}_base_roll_joint">
+          <hardwareInterface>EffortJointInterface</hardwareInterface>
+        </joint>
+        <actuator name="{side}_base_roll_motor">
+          <hardwareInterface>EffortJointInterface</hardwareInterface>
+          <mechanicalReduction>1</mechanicalReduction>
+        </actuator>
+      </transmission>
+    </xacro:if>
   </xacro:macro>
 </robot>

File: blue_descriptions/urdf/gripper_v0/gripper.urdf.xacro (robot description, xacro)
@@ -2,6 +2,5 @@
 <!-- XML namespaces -->
 <robot xmlns:xacro="http://ros.org/wiki/xacro">
-  <!-- ============================  link  ============================ -->
-  <!-- Includes elbow flex, FA roll joints in macros below -->
+  <!-- ============================  End link and gripper ============================ -->
   <xacro:macro name="blue_end_effector_v0" params="side name">
     <xacro:blue_end_v0 side="${side}" name="${name}"/>

File: blue_descriptions/urdf/robot_base_v0/robot_base.urdf.xacro (robot description, xacro)
@@ -2,10 +2,14 @@
 <!-- XML namespaces -->
 <robot xmlns:xacro="http://ros.org/wiki/xacro">
-  <!-- Inertial properties differ slightly for left vs right arm -->
-  <xacro:property name="base_camera_height"  value="0.303506965011826" />
-  <xacro:property name="camera_angle"  value= "0.0" />
-  <!-- ============================  link  ============================ -->
-  <!-- Includes elbow flex, FA roll joints in macros below -->
-  <xacro:macro name="blue_robot_base_v0" params="">
+  <!-- ============================  Robot Base  ============================ -->
+  <xacro:macro name="blue_robot_base_v0" params="cam_height cam_angle is_gazebo:=false">
+  <xacro:if value="${is_gazebo}">
+    <link name="world"/>
+    <joint name ="world_joint" type= "fixed">
+      <origin xyz="0 0 1.4" rpy="0 0 0" />
+      <parent link="world"/>
+      <child link="base_link"/>
+    </joint>
+  </xacro:if>
   <link
     name="base_link">
@@ -33,6 +37,5 @@
       </geometry>
       <material
-        name="">
-        <color
+        name=""> <color
           rgba="0.792156862745098 0.819607843137255 0.933333333333333 1" />
       </material>
@@ -118,6 +121,6 @@
     type="fixed">
     <origin
-      xyz="-0.0190500000000001 0 ${base_camera_height}"
-      rpy="1.5707963267949 -5.91437301648455E-15 ${camera_angle}" />
+      xyz="-0.0190500000000001 0 ${cam_height}"
+      rpy="1.5707963267949 -5.91437301648455E-15 ${cam_angle}" />
     <parent
       link="base_link" />

Commit message: renamed v0 to v1

File: blue_descriptions/robots/blue_full.urdf.xacro (robot description, xacro)
@@ -4,10 +4,10 @@
   <xacro:property name="is_gazebo" value="$(arg is_gazebo)" />
   <!-- ====== Load in robot base macro ====== -->
-  <xacro:include filename="$(find blue_descriptions)/urdf/robot_base_v0/robot_base.urdf.xacro" />
+  <xacro:include filename="$(find blue_descriptions)/urdf/robot_base_v1/robot_base.urdf.xacro" />
   <!-- ====== Robot camera height and angle parameters  ====== -->
   <xacro:property name="base_camera_height"  value="0.303506965011826" />
   <xacro:property name="camera_angle"  value= "0.0" />
   <!-- ====== Build base ====== -->
-  <xacro:blue_robot_base_v0 cam_height="${base_camera_height}" cam_angle="${camera_angle}" is_gazebo="${is_gazebo}"/>
+  <xacro:blue_robot_base_v1 cam_height="${base_camera_height}" cam_angle="${camera_angle}" is_gazebo="${is_gazebo}"/>
   <!-- ====== Build right and left arms====== -->
   <xacro:include filename="$(find blue_descriptions)/robots/blue_right.urdf.xacro" />

File: blue_descriptions/robots/blue_left.urdf.xacro (robot description, xacro)
@@ -3,12 +3,12 @@
   <xacro:arg name="is_gazebo" default="false" />
   <xacro:property name="is_gazebo" value="$(arg is_gazebo)" />
-  <xacro:include filename="$(find blue_descriptions)/urdf/base_v0/base.urdf.xacro" />
-  <xacro:include filename="$(find blue_descriptions)/urdf/link_v0/link.urdf.xacro" />
-  <xacro:include filename="$(find blue_descriptions)/urdf/gripper_v0/gripper.urdf.xacro" />
-  <xacro:blue_base_v0 side="left" reflect="1" child="shoulder_roll_link"/>
-  <xacro:blue_link_v0 side="left" stage="shoulder" child="elbow_roll_link" reflect="1" />
-  <xacro:blue_link_v0 side="left" stage="elbow" child="wrist_roll_link" reflect="-1" />
-  <xacro:blue_link_v0 side="left" stage="wrist" child="end_roll_link" reflect="0" wrist="1"/>
-  <xacro:blue_end_effector_v0 side="left" name="end_roll_link"/>
+  <xacro:include filename="$(find blue_descriptions)/urdf/base_v1/base.urdf.xacro" />
+  <xacro:include filename="$(find blue_descriptions)/urdf/link_v1/link.urdf.xacro" />
+  <xacro:include filename="$(find blue_descriptions)/urdf/gripper_v1/gripper.urdf.xacro" />
+  <xacro:blue_base_v1 side="left" reflect="1" child="shoulder_roll_link"/>
+  <xacro:blue_link_v1 side="left" stage="shoulder" child="elbow_roll_link" reflect="1" />
+  <xacro:blue_link_v1 side="left" stage="elbow" child="wrist_roll_link" reflect="-1" />
+  <xacro:blue_link_v1 side="left" stage="wrist" child="end_roll_link" reflect="0" wrist="1"/>
+  <xacro:blue_end_effector_v1 side="left" name="end_roll_link"/>
   <xacro:if value="${is_gazebo}">
     <gazebo>

File: blue_descriptions/robots/blue_right.urdf.xacro (robot description, xacro)
@@ -3,12 +3,12 @@
   <xacro:arg name="is_gazebo" default="false" />
   <xacro:property name="is_gazebo" value="$(arg is_gazebo)" />
-  <xacro:include filename="$(find blue_descriptions)/urdf/base_v0/base.urdf.xacro" />
-  <xacro:include filename="$(find blue_descriptions)/urdf/link_v0/link.urdf.xacro" />
-  <xacro:include filename="$(find blue_descriptions)/urdf/gripper_v0/gripper.urdf.xacro" />
-  <xacro:blue_base_v0 side="right" reflect="-1" child="shoulder_roll_link"/>
-  <xacro:blue_link_v0 side="right" stage="shoulder" child="elbow_roll_link" reflect="-1" />
-  <xacro:blue_link_v0 side="right" stage="elbow" child="wrist_roll_link" reflect="1" />
-  <xacro:blue_link_v0 side="right" stage="wrist" child="end_roll_link" reflect="0" wrist="1"/>
-  <xacro:blue_end_effector_v0 side="right" name="end_roll_link"/>
+  <xacro:include filename="$(find blue_descriptions)/urdf/base_v1/base.urdf.xacro" />
+  <xacro:include filename="$(find blue_descriptions)/urdf/link_v1/link.urdf.xacro" />
+  <xacro:include filename="$(find blue_descriptions)/urdf/gripper_v1/gripper.urdf.xacro" />
+  <xacro:blue_base_v1 side="right" reflect="-1" child="shoulder_roll_link"/>
+  <xacro:blue_link_v1 side="right" stage="shoulder" child="elbow_roll_link" reflect="-1" />
+  <xacro:blue_link_v1 side="right" stage="elbow" child="wrist_roll_link" reflect="1" />
+  <xacro:blue_link_v1 side="right" stage="wrist" child="end_roll_link" reflect="0" wrist="1"/>
+  <xacro:blue_end_effector_v1 side="right" name="end_roll_link"/>
   <xacro:if value="${is_gazebo}">
     <gazebo>

File: blue_descriptions/robots/blue_stand.urdf.xacro (robot description, xacro)
@@ -3,12 +3,12 @@
   <xacro:arg name="is_gazebo" default="false" />
   <xacro:property name="is_gazebo" value="$(arg is_gazebo)" />
-  <xacro:include filename="$(find blue_descriptions)/urdf/base_v0/base.urdf.xacro" />
-  <xacro:include filename="$(find blue_descriptions)/urdf/link_v0/link.urdf.xacro" />
-  <xacro:include filename="$(find blue_descriptions)/urdf/gripper_v0/gripper.urdf.xacro" />
-  <xacro:blue_base_v0 side="stand" reflect="-1" child="shoulder_roll_link"/>
-  <xacro:blue_link_v0 side="stand" stage="shoulder" child="elbow_roll_link" reflect="-1" />
-  <xacro:blue_link_v0 side="stand" stage="elbow" child="wrist_roll_link" reflect="1" />
-  <xacro:blue_link_v0 side="stand" stage="wrist" child="end_roll_link" reflect="0" wrist="1"/>
-  <xacro:blue_end_effector_v0 side="stand" name="end_roll_link"/>
+  <xacro:include filename="$(find blue_descriptions)/urdf/base_v1/base.urdf.xacro" />
+  <xacro:include filename="$(find blue_descriptions)/urdf/link_v1/link.urdf.xacro" />
+  <xacro:include filename="$(find blue_descriptions)/urdf/gripper_v1/gripper.urdf.xacro" />
+  <xacro:blue_base_v1 side="stand" reflect="-1" child="shoulder_roll_link"/>
+  <xacro:blue_link_v1 side="stand" stage="shoulder" child="elbow_roll_link" reflect="-1" />
+  <xacro:blue_link_v1 side="stand" stage="elbow" child="wrist_roll_link" reflect="1" />
+  <xacro:blue_link_v1 side="stand" stage="wrist" child="end_roll_link" reflect="0" wrist="1"/>
+  <xacro:blue_end_effector_v1 side="stand" name="end_roll_link"/>
   <xacro:if value="${is_gazebo}">
     <gazebo>

File: blue_descriptions/urdf/base_v1/base.urdf.xacro (robot description, xacro)
@@ -9,5 +9,5 @@
   <!-- ============================  link  ============================ -->
   <!-- Includes elbow flex, FA roll joints in macros below -->
-  <xacro:macro name="blue_base_v0" params="side reflect child">
+  <xacro:macro name="blue_base_v1" params="side reflect child">
     <link name="${side}_base_link">
       <inertial>

File: blue_descriptions/urdf/gripper_v1/gripper.urdf.xacro (robot description, xacro)
@@ -3,10 +3,10 @@
 <robot xmlns:xacro="http://ros.org/wiki/xacro">
   <!-- ============================  End link and gripper ============================ -->
-  <xacro:macro name="blue_end_effector_v0" params="side name">
-    <xacro:blue_end_v0 side="${side}" name="${name}"/>
-    <xacro:blue_gripper_v0 side="${side}" parent="${name}"/>
-    <xacro:blue_gripper_finger_v0 side="${side}" parent="${name}"/>
+  <xacro:macro name="blue_end_effector_v1" params="side name">
+    <xacro:blue_end_v1 side="${side}" name="${name}"/>
+    <xacro:blue_gripper_v1 side="${side}" parent="${name}"/>
+    <xacro:blue_gripper_finger_v1 side="${side}" parent="${name}"/>
   </xacro:macro>
-  <xacro:macro name="blue_end_v0" params="side name">
+  <xacro:macro name="blue_end_v1" params="side name">
     <link
       name="${side}_${name}">
@@ -48,5 +48,5 @@
     </link>
   </xacro:macro>
-  <xacro:macro name="blue_gripper_finger_v0" params="side parent">
+  <xacro:macro name="blue_gripper_finger_v1" params="side parent">
     <link
       name="${side}_gripper_finger_link">
@@ -64,5 +64,5 @@
     </joint>
   </xacro:macro>
-  <xacro:macro name="blue_gripper_v0" params="side parent">
+  <xacro:macro name="blue_gripper_v1" params="side parent">
     <link
       name="${side}_gripper_link">

File: blue_descriptions/urdf/link_v1/link.urdf.xacro (robot description, xacro)
@@ -4,9 +4,9 @@
   <!-- ============================  link  ============================ -->
   <!-- Includes elbow flex, FA roll joints in macros below -->
-  <xacro:macro name="blue_link_v0" params="side stage child reflect wrist:=0">
-    <xacro:blue_roll_link_v0 side="${side}" stage="${stage}" reflect="${reflect}" wrist="${wrist}"/>
-    <xacro:blue_lift_link_v0 side="${side}" stage="${stage}" child="${child}" reflect="${reflect}" />
+  <xacro:macro name="blue_link_v1" params="side stage child reflect wrist:=0">
+    <xacro:blue_roll_link_v1 side="${side}" stage="${stage}" reflect="${reflect}" wrist="${wrist}"/>
+    <xacro:blue_lift_link_v1 side="${side}" stage="${stage}" child="${child}" reflect="${reflect}" />
   </xacro:macro>
-  <xacro:macro name="blue_roll_link_v0" params="side stage reflect wrist">
+  <xacro:macro name="blue_roll_link_v1" params="side stage reflect wrist">
     <link
       name="${side}_${stage}_roll_link">
@@ -93,5 +93,5 @@
     </joint>
   </xacro:macro>
-  <xacro:macro name="blue_lift_link_v0" params="side stage child reflect">
+  <xacro:macro name="blue_lift_link_v1" params="side stage child reflect">
     <link
       name="${side}_${stage}_lift_link">

File: blue_descriptions/urdf/robot_base_v1/robot_base.urdf.xacro (robot description, xacro)
@@ -3,5 +3,5 @@
 <robot xmlns:xacro="http://ros.org/wiki/xacro">
   <!-- ============================  Robot Base  ============================ -->
-  <xacro:macro name="blue_robot_base_v0" params="cam_height cam_angle is_gazebo:=false">
+  <xacro:macro name="blue_robot_base_v1" params="cam_height cam_angle is_gazebo:=false">
   <xacro:if value="${is_gazebo}">
     <link name="world"/>
