Commit message: updated stls

File: blue_descriptions/robots/blue_full_v1.urdf.xacro (robot description, xacro)
@@ -11,5 +11,5 @@
   <xacro:blue_robot_base_v1 cam_height="${base_camera_height}" cam_angle="${camera_angle}" is_gazebo="${is_gazebo}"/>
   <!-- ====== Build right and left arms====== -->
-  <xacro:include filename="$(find blue_descriptions)/robots/blue_right.urdf.xacro" />
-  <xacro:include filename="$(find blue_descriptions)/robots/blue_left.urdf.xacro" />
+  <xacro:include filename="$(find blue_descriptions)/robots/blue_right_v1.urdf.xacro" />
+  <xacro:include filename="$(find blue_descriptions)/robots/blue_left_v1.urdf.xacro" />
 </robot>

File: blue_descriptions/urdf/base_v1/base.urdf.xacro (robot description, xacro)
@@ -31,5 +31,5 @@
         <geometry>
           <mesh
-            filename="package://blue_descriptions/meshes/arm_base_link.STL" />
+            filename="package://blue_descriptions/meshes/arm_base_link_v1.STL" />
         </geometry>
         <material name="">
@@ -43,5 +43,5 @@
         <geometry>
           <mesh
-            filename="package://blue_descriptions/meshes/arm_base_link.STL" />
+            filename="package://blue_descriptions/meshes/arm_base_link_v1.STL" />
         </geometry>
       </collision>

File: blue_descriptions/urdf/base_v2/base.urdf.xacro (robot description, xacro)
@@ -32,5 +32,5 @@
         <geometry>
           <mesh
-            filename="package://blue_descriptions/meshes/arm_base_link.STL" />
+            filename="package://blue_descriptions/meshes/arm_base_link_v2.STL" />
         </geometry>
         <material name="">
@@ -44,5 +44,5 @@
         <geometry>
           <mesh
-            filename="package://blue_descriptions/meshes/arm_base_link.STL" />
+            filename="package://blue_descriptions/meshes/arm_base_link_v2.STL" />
         </geometry>
       </collision>

File: blue_descriptions/urdf/link_v1/link.urdf.xacro (robot description, xacro)
@@ -31,5 +31,5 @@
         <geometry>
           <mesh
-            filename="package://blue_descriptions/meshes/roll_link.STL" />
+            filename="package://blue_descriptions/meshes/roll_link_v1.STL" />
         </geometry>
         <material name="">
@@ -43,5 +43,5 @@
         <geometry>
           <mesh
-            filename="package://blue_descriptions/meshes/roll_link.STL" />
+            filename="package://blue_descriptions/meshes/roll_link_v1.STL" />
         </geometry>
       </collision>
@@ -116,5 +116,5 @@
         <geometry>
           <mesh
-            filename="package://blue_descriptions/meshes/lift_link.STL" />
+            filename="package://blue_descriptions/meshes/lift_link_v1.STL" />
         </geometry>
         <material name="">
@@ -128,5 +128,5 @@
         <geometry>
           <mesh
-            filename="package://blue_descriptions/meshes/lift_link.STL" />
+            filename="package://blue_descriptions/meshes/lift_link_v1.STL" />
         </geometry>
       </collision>

File: blue_descriptions/urdf/link_v2/link.urdf.xacro (robot description, xacro)
@@ -4,24 +4,24 @@
   <!-- ============================  link  ============================ -->
   <!-- Includes elbow flex, FA roll joints in macros below -->
-  <xacro:macro name="blue_link_v1" params="side stage child reflect wrist:=0">
-    <xacro:blue_roll_link_v1 side="${side}" stage="${stage}" reflect="${reflect}" wrist="${wrist}"/>
-    <xacro:blue_lift_link_v1 side="${side}" stage="${stage}" child="${child}" reflect="${reflect}" />
+  <xacro:macro name="blue_link_v2" params="side stage child reflect wrist:=0">
+    <xacro:blue_roll_link_v2 side="${side}" stage="${stage}" reflect="${reflect}" wrist="${wrist}"/>
+    <xacro:blue_lift_link_v2 side="${side}" stage="${stage}" child="${child}" reflect="${reflect}" />
   </xacro:macro>
-  <xacro:macro name="blue_roll_link_v1" params="side stage reflect wrist">
+  <xacro:macro name="blue_roll_link_v2" params="side stage reflect wrist">
     <link
       name="${side}_${stage}_roll_link">
       <inertial>
         <origin
-          xyz="0.00526385736219506 2.70691865020822E-05 -0.0641638075944594"
+          xyz="2.96915144581966E-07 -0.00817928723072138 0.120962910647003"
           rpy="0 0 0" />
         <mass
-          value="${1.91396434922939 - 0.50028 * wrist}" />
+          value="0.37905420680448" />
         <inertia
-          ixx="0.0057866591250737"
-          ixy="3.71515699629511E-07"
-          ixz="-6.32890111626103E-05"
-          iyy="0.00530223654324281"
-          iyz="8.9999884666805E-07"
-          izz="0.00342399181200673" />
+          ixx="0.00156534155265803"
+          ixy="7.86255262568044E-09"
+          ixz="1.53529042690406E-08"
+          iyy="0.00178123169436239"
+          iyz="1.62349609777295E-06"
+          izz="0.000959456942468469" />
       </inertial>
       <visual>
@@ -31,5 +31,5 @@
         <geometry>
           <mesh
-            filename="package://blue_descriptions/meshes/roll_link.STL" />
+            filename="package://blue_descriptions/meshes/roll_link_v2.STL" />
         </geometry>
         <material name="">
@@ -43,5 +43,5 @@
         <geometry>
           <mesh
-            filename="package://blue_descriptions/meshes/roll_link.STL" />
+            filename="package://blue_descriptions/meshes/roll_link_v2.STL" />
         </geometry>
       </collision>
@@ -51,6 +51,6 @@
       type="revolute">
       <origin
-        xyz="-0.01143 0 -0.18056"
-        rpy="-1.5708 4.4409E-16 3.1416" />
+        xyz="0 0.012 0.23278"
+        rpy="1.5708 4.9887E-16 -1.5708" />
       <parent
         link="${side}_${stage}_roll_link"/>
@@ -93,20 +93,20 @@
     </joint>
   </xacro:macro>
-  <xacro:macro name="blue_lift_link_v1" params="side stage child reflect">
+  <xacro:macro name="blue_lift_link_v2" params="side stage child reflect">
     <link
       name="${side}_${stage}_lift_link">
       <inertial>
         <origin
-          xyz="-5.0083559080677E-06 0.000232928456050885 -1.77451392545103E-05"
+          xyz="-3.66305969445868E-08 -0.000820052992464293 -6.62529991840577E-08"
           rpy="0 0 0" />
         <mass
-          value="0.448307108622636" />
+          value="1.02342370509176" />
         <inertia
-          ixx="0.000804272985961788"
-          ixy="4.84548777859872E-08"
-          ixz="2.09160815704306E-06"
-          iyy="0.000818260636171894"
-          iyz="-1.44954778549764E-08"
-          izz="0.000550840705045094" />
+          ixx="0.00185674588732204"
+          ixy="2.50286442134684E-09"
+          ixz="-3.11007993614261E-09"
+          iyy="0.00185731655609116"
+          iyz="2.89693722882194E-09"
+          izz="0.00152396319769825" />
       </inertial>
       <visual>
@@ -116,5 +116,5 @@
         <geometry>
           <mesh
-            filename="package://blue_descriptions/meshes/lift_link.STL" />
+            filename="package://blue_descriptions/meshes/lift_link_v2.STL" />
         </geometry>
         <material name="">
@@ -128,5 +128,5 @@
         <geometry>
           <mesh
-            filename="package://blue_descriptions/meshes/lift_link.STL" />
+            filename="package://blue_descriptions/meshes/lift_link_v2.STL" />
         </geometry>
       </collision>
@@ -136,6 +136,6 @@
       type="revolute">
       <origin
-        xyz="0 0.070147 -6.25E-05"
-        rpy="-1.5708 ${reflect*1.5673} -3.1416" />
+        xyz="0 0.035953 0"
+        rpy="1.5708 -3.8798E-16 -3.1416" />
       <parent
         link="${side}_${stage}_lift_link"/>

Commit message: updated urdf to allow for base_link=={side}_base_link for single arm setups

File: blue_descriptions/robots/blue_full_v1.urdf.xacro (robot description, xacro)
@@ -3,4 +3,6 @@
   <xacro:arg name="is_gazebo" default="false" />
   <xacro:property name="is_gazebo" value="$(arg is_gazebo)" />
+  <xacro:arg name="set_base_link" default="false" />
+  <xacro:property name="set_base_link" value="$(arg set_base_link)" />
   <!-- ====== Load in robot base macro ====== -->
   <xacro:include filename="$(find blue_descriptions)/urdf/robot_base_v1/robot_base.urdf.xacro" />

File: blue_descriptions/robots/blue_full_v2.urdf.xacro (robot description, xacro)
@@ -3,4 +3,6 @@
   <xacro:arg name="is_gazebo" default="false" />
   <xacro:property name="is_gazebo" value="$(arg is_gazebo)" />
+  <xacro:arg name="set_base_link" default="false" />
+  <xacro:property name="set_base_link" value="$(arg set_base_link)" />
   <!-- ====== Load in robot base macro ====== -->
   <xacro:include filename="$(find blue_descriptions)/urdf/robot_base_v1/robot_base.urdf.xacro" />

File: blue_descriptions/robots/blue_left_v1.urdf.xacro (robot description, xacro)
@@ -3,4 +3,24 @@
   <xacro:arg name="is_gazebo" default="false" />
   <xacro:property name="is_gazebo" value="$(arg is_gazebo)" />
+  <xacro:arg name="set_base_link" default="true" />
+  <xacro:property name="set_base_link" value="$(arg set_base_link)" />
+  <xacro:if value="${set_base_link}">
+    <link
+      name="base_link">
+    </link>
+    <joint
+      name="left_fixed_joint"
+      type="fixed">
+      <origin
+        xyz="0.0 0.0 0.0"
+        rpy="0.0 0.0 0.0" />
+      <parent
+        link="base_link" />
+      <child
+        link="left_base_link" />
+      <axis
+        xyz="0.0 0.0 0.0" />
+    </joint>
+  </xacro:if>
   <xacro:include filename="$(find blue_descriptions)/urdf/base_v1/base.urdf.xacro" />
   <xacro:include filename="$(find blue_descriptions)/urdf/link_v1/link.urdf.xacro" />

File: blue_descriptions/robots/blue_left_v2.urdf.xacro (robot description, xacro)
@@ -3,4 +3,24 @@
   <xacro:arg name="is_gazebo" default="false" />
   <xacro:property name="is_gazebo" value="$(arg is_gazebo)" />
+  <xacro:arg name="set_base_link" default="true" />
+  <xacro:property name="set_base_link" value="$(arg set_base_link)" />
+  <xacro:if value="${set_base_link}">
+    <link
+      name="base_link">
+    </link>
+    <joint
+      name="left_fixed_joint"
+      type="fixed">
+      <origin
+        xyz="0.0 0.0 0.0"
+        rpy="0.0 0.0 0.0" />
+      <parent
+        link="base_link" />
+      <child
+        link="left_base_link" />
+      <axis
+        xyz="0.0 0.0 0.0" />
+    </joint>
+  </xacro:if>
   <xacro:include filename="$(find blue_descriptions)/urdf/base_v2/base.urdf.xacro" />
   <xacro:include filename="$(find blue_descriptions)/urdf/link_v2/link.urdf.xacro" />

File: blue_descriptions/robots/blue_right_v1.urdf.xacro (robot description, xacro)
@@ -3,4 +3,24 @@
   <xacro:arg name="is_gazebo" default="false" />
   <xacro:property name="is_gazebo" value="$(arg is_gazebo)" />
+  <xacro:arg name="set_base_link" default="true" />
+  <xacro:property name="set_base_link" value="$(arg set_base_link)" />
+  <xacro:if value="${set_base_link}">
+    <link
+      name="base_link">
+    </link>
+    <joint
+      name="right_fixed_joint"
+      type="fixed">
+      <origin
+        xyz="0.0 0.0 0.0"
+        rpy="0.0 0.0 0.0" />
+      <parent
+        link="base_link" />
+      <child
+        link="right_base_link" />
+      <axis
+        xyz="0.0 0.0 0.0" />
+    </joint>
+  </xacro:if>
   <xacro:include filename="$(find blue_descriptions)/urdf/base_v1/base.urdf.xacro" />
   <xacro:include filename="$(find blue_descriptions)/urdf/link_v1/link.urdf.xacro" />

File: blue_descriptions/robots/blue_right_v2.urdf.xacro (robot description, xacro)
@@ -3,4 +3,24 @@
   <xacro:arg name="is_gazebo" default="false" />
   <xacro:property name="is_gazebo" value="$(arg is_gazebo)" />
+  <xacro:arg name="set_base_link" default="true" />
+  <xacro:property name="set_base_link" value="$(arg set_base_link)" />
+  <xacro:if value="${set_base_link}">
+    <link
+      name="base_link">
+    </link>
+    <joint
+      name="right_fixed_joint"
+      type="fixed">
+      <origin
+        xyz="0.0 0.0 0.0"
+        rpy="0.0 0.0 0.0" />
+      <parent
+        link="base_link" />
+      <child
+        link="right_base_link" />
+      <axis
+        xyz="0.0 0.0 0.0" />
+    </joint>
+  </xacro:if>
   <xacro:include filename="$(find blue_descriptions)/urdf/base_v2/base.urdf.xacro" />
   <xacro:include filename="$(find blue_descriptions)/urdf/link_v2/link.urdf.xacro" />
