Commit message: cleaned up Joint position controller, fixed some xacros formatting

File: blue_descriptions/urdf/base_v0/base.urdf.xacro (robot description, xacro)
@@ -33,8 +33,6 @@
             filename="package://blue_descriptions/meshes/arm_base_link.STL" />
         </geometry>
-        <material
-          name="">
-          <color
-            rgba="0.792156862745098 0.819607843137255 0.933333333333333 1" />
+        <material name="">
+          <color rgba="0.792156862745098 0.819607843137255 0.933333333333333 1" />
         </material>
       </visual>
@@ -64,6 +62,6 @@
         lower="${0.5*((reflect+1)*base_left_min+(1-reflect)*base_right_min)}"
         upper="${0.5*((reflect+1)*base_left_max+(1-reflect)*base_right_max)}"
-        effort="30"
-        velocity="20" />
+        effort="80"
+        velocity="50" />
     </joint>
     <xacro:if value="${is_gazebo}">

File: blue_descriptions/urdf/gripper_v0/gripper.urdf.xacro (robot description, xacro)
@@ -32,8 +32,6 @@
             filename="package://blue_descriptions/meshes/wrist_roll_link.STL" />
         </geometry>
-        <material
-          name="">
-          <color
-            rgba="1 1 1 1" />
+        <material name="">
+          <color rgba="1 1 1 1" />
         </material>
       </visual>
@@ -105,6 +103,6 @@
         lower="-2.6761"
         upper="2.6761"
-        effort="30"
-        velocity="20" />
+        effort="80"
+        velocity="50" />
     </joint>
     <xacro:if value="${is_gazebo}">

File: blue_descriptions/urdf/link_v0/link.urdf.xacro (robot description, xacro)
@@ -33,8 +33,6 @@
             filename="package://blue_descriptions/meshes/roll_link.STL" />
         </geometry>
-        <material
-          name="">
-          <color
-            rgba="1 1 1 1" />
+        <material name="">
+          <color rgba="1 1 1 1" />
         </material>
       </visual>
@@ -64,6 +62,6 @@
         lower="-2.2944"
         upper="0"
-        effort="30"
-        velocity="20" />
+        effort="80"
+        velocity="50" />
     </joint>
     <xacro:if value="${is_gazebo}">
@@ -105,8 +103,6 @@
             filename="package://blue_descriptions/meshes/lift_link.STL" />
         </geometry>
-        <material
-          name="">
-          <color
-            rgba="0.792156862745098 0.819607843137255 0.933333333333333 1" />
+        <material name="">
+          <color rgba="0.116747 0.862745 1.0 1" />
         </material>
       </visual>
@@ -136,6 +132,6 @@
         lower="-2.6761"
         upper="2.6761"
-        effort="30"
-        velocity="20" />
+        effort="80"
+        velocity="50" />
     </joint>
     <xacro:if value="${is_gazebo}">

File: blue_descriptions/urdf/robot_base_v0/robot_base.urdf.xacro (robot description, xacro)
@@ -36,7 +36,6 @@
           filename="package://blue_descriptions/meshes/robot_base_link.STL" />
       </geometry>
-      <material
-        name=""> <color
-          rgba="0.792156862745098 0.819607843137255 0.933333333333333 1" />
+      <material name="">
+        <color rgba="0.792156862745098 0.819607843137255 0.933333333333333 1" />
       </material>
     </visual>
@@ -101,8 +100,6 @@
           filename="package://blue_descriptions/meshes/camera_link.STL" />
       </geometry>
-      <material
-        name="">
-        <color
-          rgba="0.792156862745098 0.819607843137255 0.933333333333333 1" />
+      <material name="">
+        <color rgba="0.792156862745098 0.819607843137255 0.933333333333333 1" />
       </material>
     </visual>
