Commit message: description update

File: blue_descriptions/urdf/gripper_v0/gripper.urdf.xacro (robot description, xacro)
@@ -6,4 +6,5 @@
     <xacro:blue_end_v0 side="${side}" name="${name}"/>
     <xacro:blue_gripper_v0 side="${side}" parent="${name}"/>
+    <xacro:blue_gripper_finger_v0 side="${side}" parent="${name}"/>
   </xacro:macro>
   <xacro:macro name="blue_end_v0" params="side name">
@@ -47,4 +48,20 @@
     </link>
   </xacro:macro>
+  <xacro:macro name="blue_gripper_finger_v0" params="side parent">
+    <link
+      name="${side}_gripper_finger_link">
+    </link>
+    <joint
+      name="${side}_gripper_finger_joint"
+      type="fixed">
+      <origin
+        xyz="0 0.0 -0.18"
+        rpy="-3.14159 -0.0 1.5708" />
+      <parent
+        link="${side}_${parent}" />
+      <child
+        link="${side}_gripper_finger_link" />
+    </joint>
+  </xacro:macro>
   <xacro:macro name="blue_gripper_v0" params="side parent">
     <link
@@ -64,27 +81,4 @@
           izz="0.000293333065172452" />
       </inertial>
-      <visual>
-        <origin
-          xyz="0 0 0"
-          rpy="0 0 0" />
-        <geometry>
-          <mesh
-            filename="package://blue_descriptions/meshes/wrist_roll_link.STL" />
-        </geometry>
-        <material
-          name="">
-          <color
-            rgba="0.792156862745098 0.819607843137255 0.933333333333333 1" />
-        </material>
-      </visual>
-      <collision>
-        <origin
-          xyz="0 0 0"
-          rpy="0 0 0" />
-        <geometry>
-          <mesh
-            filename="package://blue_descriptions/meshes/wrist_roll_link.STL" />
-        </geometry>
-      </collision>
     </link>
     <joint

Commit message: added mimic joints for individual fingers

File: blue_descriptions/urdf/gripper_v0/gripper.urdf.xacro (robot description, xacro)
@@ -95,6 +95,6 @@
         xyz="0 0 1" />
       <limit
-        lower="-2.6761"
-        upper="2.6761"
+        lower="0"
+        upper="1.05"
         effort="800"
         velocity="50" />
@@ -112,4 +112,230 @@
       </transmission>
     </xacro:if>
+    <!-- right finger -->
+    <link
+      name="${side}_r_finger_link">
+      <inertial>
+        <origin
+          xyz="0.00046733152633803 0.0122666320844707 1.16452530510985E-07"
+          rpy="0 0 0" />
+        <mass
+          value="0.0384620979765985" />
+        <inertia
+          ixx="1.93716279065148E-05"
+          ixy="-1.74835869619804E-06"
+          ixz="3.21020594362941E-11"
+          iyy="5.23390911087335E-06"
+          iyz="-5.04535602261134E-11"
+          izz="1.92560542157392E-05" />
+      </inertial>
+      <visual>
+        <origin
+          xyz="0 0 0"
+          rpy="0 0 0" />
+        <geometry>
+          <mesh
+            filename="package://blue_descriptions/meshes/finger_limb_link.STL" />
+        </geometry>
+        <material
+          name="">
+          <color
+            rgba="0.792156862745098 0.819607843137255 0.933333333333333 1" />
+        </material>
+      </visual>
+      <collision>
+        <origin
+          xyz="0 0 0"
+          rpy="0 0 0" />
+        <geometry>
+          <mesh
+            filename="package://blue_descriptions/meshes/finger_limb_link.STL" />
+        </geometry>
+      </collision>
+    </link>
+    <joint
+      name="${side}_r_finger_joint"
+      type="continuous">
+      <origin
+        xyz="0.000 0.030703 -0.071979"
+        rpy="-1.5708 -0.63969 1.5708" />
+      <parent
+        link="${side}_${parent}" />
+      <child
+        link="${side}_r_finger_link" />
+      <axis
+        xyz="0 0 1" />
+      <mimic
+        joint="${side}_gripper_joint"
+        multiplier="1"/>
+    </joint>
+    <link
+      name="${side}_r_finger_tip_link">
+      <inertial>
+        <origin
+          xyz="0.000428096363398578 -6.3962924111774E-08 0.0162809660053768"
+          rpy="0 0 0" />
+        <mass
+          value="0.0096424502794395" />
+        <inertia
+          ixx="1.76146900164229E-06"
+          ixy="-1.63725174281941E-11"
+          ixz="-5.09403577370148E-07"
+          iyy="1.95368501856251E-06"
+          iyz="-2.7403586363238E-12"
+          izz="6.78506827465793E-07" />
+      </inertial>
+      <visual>
+        <origin
+          xyz="0 0 0"
+          rpy="0 0 0" />
+        <geometry>
+          <mesh
+            filename="package://blue_descriptions/meshes/finger_tip_link.STL" />
+        </geometry>
+        <material
+          name="">
+          <color
+            rgba="0.792156862745098 0.819607843137255 0.933333333333333 1" />
+        </material>
+      </visual>
+      <collision>
+        <origin
+          xyz="0 0 0"
+          rpy="0 0 0" />
+        <geometry>
+          <mesh
+            filename="package://blue_descriptions/meshes/finger_tip_link.STL" />
+        </geometry>
+      </collision>
+    </link>
+    <joint
+      name="${side}_r_finger_tip_joint"
+      type="continuous">
+      <origin
+        xyz="0 0.06 0"
+        rpy="1.5708 -1.5754E-31 -2.5019" />
+      <parent
+        link="${side}_r_finger_link" />
+      <child
+        link="${side}_r_finger_tip_link" />
+      <axis
+        xyz="0 1 0" />
+      <mimic
+        joint="${side}_gripper_joint"
+        multiplier="-1"/>
+    </joint>
+    <!-- left finger -->
+    <link
+      name="${side}_l_finger_link">
+      <inertial>
+        <origin
+          xyz="0.00046733152633803 0.0122666320844707 1.16452530510985E-07"
+          rpy="0 0 0" />
+        <mass
+          value="0.0384620979765985" />
+        <inertia
+          ixx="1.93716279065148E-05"
+          ixy="-1.74835869619804E-06"
+          ixz="3.21020594362941E-11"
+          iyy="5.23390911087335E-06"
+          iyz="-5.04535602261134E-11"
+          izz="1.92560542157392E-05" />
+      </inertial>
+      <visual>
+        <origin
+          xyz="0 0 0"
+          rpy="0 0 0" />
+        <geometry>
+          <mesh
+            filename="package://blue_descriptions/meshes/finger_limb_link.STL" />
+        </geometry>
+        <material
+          name="">
+          <color
+            rgba="0.792156862745098 0.819607843137255 0.933333333333333 1" />
+        </material>
+      </visual>
+      <collision>
+        <origin
+          xyz="0 0 0"
+          rpy="0 0 0" />
+        <geometry>
+          <mesh
+            filename="package://blue_descriptions/meshes/finger_limb_link.STL" />
+        </geometry>
+      </collision>
+    </link>
+    <joint
+      name="${side}_l_finger_joint"
+      type="continuous">
+      <origin
+        xyz="0.000 -0.030703 -0.071979"
+        rpy="-1.5708 -0.63969 -1.5708" />
+      <parent
+        link="${side}_${parent}" />
+      <child
+        link="${side}_l_finger_link" />
+      <axis
+        xyz="0 0 1" />
+      <mimic
+        joint="${side}_gripper_joint"
+        multiplier="1"/>
+    </joint>
+    <link
+      name="${side}_l_finger_tip_link">
+      <inertial>
+        <origin
+          xyz="0.000428096363398578 -6.3962924111774E-08 0.0162809660053768"
+          rpy="0 0 0" />
+        <mass
+          value="0.0096424502794395" />
+        <inertia
+          ixx="1.76146900164229E-06"
+          ixy="-1.63725174281941E-11"
+          ixz="-5.09403577370148E-07"
+          iyy="1.95368501856251E-06"
+          iyz="-2.7403586363238E-12"
+          izz="6.78506827465793E-07" />
+      </inertial>
+      <visual>
+        <origin
+          xyz="0 0 0"
+          rpy="0 0 0" />
+        <geometry>
+          <mesh
+            filename="package://blue_descriptions/meshes/finger_tip_link.STL" />
+        </geometry>
+        <material
+          name="">
+          <color
+            rgba="0.792156862745098 0.819607843137255 0.933333333333333 1" />
+        </material>
+      </visual>
+      <collision>
+        <origin
+          xyz="0 0 0"
+          rpy="0 0 0" />
+        <geometry>
+          <mesh
+            filename="package://blue_descriptions/meshes/finger_tip_link.STL" />
+        </geometry>
+      </collision>
+    </link>
+    <joint
+      name="${side}_l_finger_tip_joint"
+      type="continuous">
+      <origin
+        xyz="0 0.06 0"
+        rpy="1.5708 -1.5754E-31 -2.5019" />
+      <parent
+        link="${side}_l_finger_link" />
+      <child
+        link="${side}_l_finger_tip_link" />
+      <axis
+        xyz="0 1 0" />
+      <mimic
+        joint="${side}_gripper_joint"
+        multiplier="-1"/>
+    </joint>
   </xacro:macro>
 </robot>
