Commit message: updated new limits and inertias

File: blue_descriptions/urdf/base_v2/base.urdf.xacro (robot description, xacro)
@@ -3,8 +3,8 @@
 <robot xmlns:xacro="http://ros.org/wiki/xacro">
   <!-- Inertial properties differ slightly for left vs right arm -->
-  <xacro:property name="base_left_min"  value="-2.3412" />
-  <xacro:property name="base_left_max"  value= "3.3999" />
-  <xacro:property name="base_right_min"  value="-3.3999" />
-  <xacro:property name="base_right_max"  value= "2.3412" />
+  <xacro:property name="base_left_min"  value="-3.14159" />
+  <xacro:property name="base_left_max"  value="3.1" />
+  <xacro:property name="base_right_min"  value="-3.1" />
+  <xacro:property name="base_right_max"  value="3.14159" />
   <!-- ============================  link  ============================ -->
   <!-- Includes elbow flex, FA roll joints in macros below -->

File: blue_descriptions/urdf/link_v2/link.urdf.xacro (robot description, xacro)
@@ -16,11 +16,11 @@
           rpy="0 0 0" />
         <mass
-          value="${1.83492 - 0.50028 * wrist}" />
+          value="${1.83492 - 0.36982 * wrist}" />
         <inertia
           ixx="61495.01E-07"
-          ixy="-19.97E-07"
-          ixz="328.6E-07"
-          iyy="50978.6E-07"
-          iyz="243.21E-07"
+          ixy="-19.9700E-07"
+          ixz="328.6000E-07"
+          iyy="50978.60E-07"
+          iyz="243.2100E-07"
           izz="41841.05E-07" />
       </inertial>
@@ -98,15 +98,15 @@
       <inertial>
         <origin
-          xyz="0.0 0.00127 0.0"
+          xyz="0.0 0.01524 0.0"
           rpy="0 0 0" />
         <mass
-          value="0.58967" />
+          value="${0.58967 - 0.14061 * wrist}" />
         <inertia
-          ixx="0.000835910502384406"
-          ixy="2.36578561626853E-07"
-          ixz="2.13858156359985E-06"
-          iyy="0.000846892587114994"
-          iyz="1.23149095856232E-07"
-          izz="0.000571368010807835" />
+          ixx="11631.35E-07"
+          ixy="0.000000E-07"
+          ixz="0.000000E-07"
+          iyy="9852.210E-07"
+          iyz="0.000000E-07"
+          izz="8916.610E-07" />
       </inertial>
       <visual>

Commit message: Add friction to links

File: blue_descriptions/urdf/base_v2/base.urdf.xacro (robot description, xacro)
@@ -51,4 +51,5 @@
       name="${side}_base_roll_joint"
       type="revolute">
+          <dynamics damping="0.7" friction="10.0"/>
       <origin
         xyz="0 0 0.0834989807730001"
@@ -70,4 +71,5 @@
         <type>transmission_interface/SimpleTransmission</type>
         <joint name="${side}_base_roll_joint">
+          <dynamics damping="0.7" friction="10.0"/>
           <hardwareInterface>hardware_interface/EffortJointInterface</hardwareInterface>
         </joint>

File: blue_descriptions/urdf/gripper_v1/gripper.urdf.xacro (robot description, xacro)
@@ -67,4 +67,5 @@
       name="${side}_gripper_finger_joint"
       type="fixed">
+        <dynamics damping="0.7" friction="10.0"/>
       <origin
         xyz="0 0.0 -0.18"
@@ -97,4 +98,5 @@
       name="${side}_gripper_joint"
       type="revolute">
+        <dynamics damping="0.7" friction="10.0"/>
       <origin
         xyz="0 0 -0.10"
@@ -116,4 +118,5 @@
         <type>transmission_interface/SimpleTransmission</type>
         <joint name="${side}_gripper_joint">
+        <dynamics damping="0.7" friction="10.0"/>
           <hardwareInterface>hardware_interface/EffortJointInterface</hardwareInterface>
         </joint>
@@ -169,4 +172,5 @@
       name="${side}_r_finger_joint"
       type="continuous">
+        <dynamics damping="0.7" friction="10.0"/>
       <origin
         xyz="0.000 0.030703 -0.071979"
@@ -225,4 +229,5 @@
       name="${side}_r_finger_tip_joint"
       type="continuous">
+        <dynamics damping="0.7" friction="10.0"/>
       <origin
         xyz="0 0.06 0"
@@ -282,4 +287,5 @@
       name="${side}_l_finger_joint"
       type="continuous">
+        <dynamics damping="0.7" friction="10.0"/>
       <origin
         xyz="0.000 -0.030703 -0.071979"

File: blue_descriptions/urdf/link_v2/link.urdf.xacro (robot description, xacro)
@@ -50,4 +50,5 @@
       name="${side}_${stage}_lift_joint"
       type="revolute">
+        <dynamics damping="0.7" friction="10.0"/>
       <origin
         xyz="-0.012 0 -0.232779056600415"
@@ -69,4 +70,5 @@
         <type>transmission_interface/SimpleTransmission</type>
         <joint name="${side}_${stage}_lift_joint">
+          <dynamics damping="0.7" friction="10.0"/>
           <hardwareInterface>hardware_interface/EffortJointInterface</hardwareInterface>
         </joint>
@@ -82,4 +84,5 @@
       name="${side}_${stage}_accel_joint"
       type="fixed">
+        <dynamics damping="0.7" friction="10.0"/>
       <origin
         xyz="-0.020008330615085 -0.000510000000000066 -0.111067108096273"
@@ -135,4 +138,5 @@
       name="${side}_${stage}_roll_joint"
       type="revolute">
+        <dynamics damping="0.7" friction="10.0"/>
       <origin
         xyz="0 ${0.0359531521130187+wrist*0.03419} 0"
@@ -154,4 +158,5 @@
         <type>transmission_interface/SimpleTransmission</type>
         <joint name="${side}_${stage}_roll_joint">
+        <dynamics damping="0.7" friction="10.0"/>
           <hardwareInterface>hardware_interface/EffortJointInterface</hardwareInterface>
         </joint>

Commit message: Resolve indentation issues

File: blue_descriptions/urdf/base_v2/base.urdf.xacro (robot description, xacro)
@@ -51,5 +51,5 @@
       name="${side}_base_roll_joint"
       type="revolute">
-          <dynamics damping="0.7" friction="10.0"/>
+      <dynamics damping="0.7" friction="10.0"/>
       <origin
         xyz="0 0 0.0834989807730001"

File: blue_descriptions/urdf/gripper_v1/gripper.urdf.xacro (robot description, xacro)
@@ -73,5 +73,5 @@
       name="${side}_gripper_finger_joint"
       type="fixed">
-        <dynamics damping="0.7" friction="10.0"/>
+      <dynamics damping="0.7" friction="10.0"/>
       <origin
         xyz="0 0.0 -0.18"
@@ -177,5 +177,5 @@
       name="${side}_r_finger_joint"
       type="continuous">
-        <dynamics damping="0.7" friction="10.0"/>
+      <dynamics damping="0.7" friction="10.0"/>
       <origin
         xyz="0.000 0.030703 -0.071979"
@@ -250,9 +250,9 @@
       <axis
         xyz="0 1 0" />
-        <mimic
-          joint="${side}_gripper_joint"
-          multiplier="-0.25"
-          offset="0.85"
-          max_effort="5"/>
+      <mimic
+        joint="${side}_gripper_joint"
+        multiplier="-0.25"
+        offset="0.85"
+        max_effort="5"/>
     </joint>
     <xacro:if value="${is_gazebo}">
@@ -305,5 +305,5 @@
       name="${side}_l_finger_joint"
       type="continuous">
-        <dynamics damping="0.7" friction="10.0"/>
+      <dynamics damping="0.7" friction="10.0"/>
       <origin
         xyz="0.000 -0.030703 -0.071979"
@@ -378,9 +378,9 @@
       <axis
         xyz="0 1 0" />
-        <mimic
-          joint="${side}_gripper_joint"
-          multiplier="-0.25"
-          offset="0.85"
-          max_effort="5"/>
+      <mimic
+        joint="${side}_gripper_joint"
+        multiplier="-0.25"
+        offset="0.85"
+        max_effort="5"/>
     </joint>
     <xacro:if value="${is_gazebo}">

File: blue_descriptions/urdf/link_v2/link.urdf.xacro (robot description, xacro)
@@ -50,5 +50,5 @@
       name="${side}_${stage}_lift_joint"
       type="revolute">
-        <dynamics damping="0.7" friction="10.0"/>
+      <dynamics damping="0.7" friction="10.0"/>
       <origin
         xyz="-0.012 0 -0.232779056600415"
@@ -84,5 +84,5 @@
       name="${side}_${stage}_accel_joint"
       type="fixed">
-        <dynamics damping="0.7" friction="10.0"/>
+      <dynamics damping="0.7" friction="10.0"/>
       <origin
         xyz="-0.020008330615085 -0.000510000000000066 -0.111067108096273"
@@ -138,5 +138,5 @@
       name="${side}_${stage}_roll_joint"
       type="revolute">
-        <dynamics damping="0.7" friction="10.0"/>
+      <dynamics damping="0.7" friction="10.0"/>
       <origin
         xyz="0 ${0.0359531521130187+wrist*0.03419} 0"
