Commit message: gripper update

File: blue_descriptions/urdf/gripper_v1/gripper.urdf.xacro (robot description, xacro)
@@ -31,5 +31,5 @@
         <geometry>
           <mesh
-            filename="package://blue_descriptions/meshes/wrist_roll_link.STL" />
+            filename="package://blue_descriptions/meshes/hand_base_link.STL" />
         </geometry>
         <material name="">
@@ -43,5 +43,5 @@
         <geometry>
           <mesh
-            filename="package://blue_descriptions/meshes/wrist_roll_link.STL" />
+            filename="package://blue_descriptions/meshes/hand_base_link.STL" />
         </geometry>
       </collision>
@@ -112,4 +112,5 @@
       </transmission>
     </xacro:if>
+    <xacro:if value="${is_gazebo == 'false'}">
     <!-- right finger -->
     <link
@@ -338,4 +339,5 @@
         multiplier="-1"/>
     </joint>
+    </xacro:if>
   </xacro:macro>
 </robot>

File: blue_descriptions/urdf/link_v2/link.urdf.xacro (robot description, xacro)
@@ -6,5 +6,5 @@
   <xacro:macro name="blue_link_v2" params="side stage child reflect wrist:=0">
     <xacro:blue_roll_link_v2 side="${side}" stage="${stage}" reflect="${reflect}" wrist="${wrist}"/>
-    <xacro:blue_lift_link_v2 side="${side}" stage="${stage}" child="${child}" reflect="${reflect}" />
+    <xacro:blue_lift_link_v2 side="${side}" stage="${stage}" child="${child}" reflect="${reflect}" wrist="${wrist}"/>
   </xacro:macro>
   <xacro:macro name="blue_roll_link_v2" params="side stage reflect wrist">
@@ -16,5 +16,5 @@
           rpy="0 0 0" />
         <mass
-          value="0.37905420680448" />
+          value="${1.91396434922939 - 0.50028 * wrist}" />
         <inertia
           ixx="0.00156534155265803"
@@ -93,5 +93,5 @@
     </joint>
   </xacro:macro>
-  <xacro:macro name="blue_lift_link_v2" params="side stage child reflect">
+  <xacro:macro name="blue_lift_link_v2" params="side stage child reflect wrist">
     <link
       name="${side}_${stage}_lift_link">
@@ -136,5 +136,5 @@
       type="revolute">
       <origin
-        xyz="0 0.0359531521130187 0"
+        xyz="0 ${0.0359531521130187+wrist*0.03419} 0"
         rpy="1.5707963267949 ${reflect*-1.56798} 0" />
       <parent

Commit message: finished gazebo support

File: blue_descriptions/urdf/gripper_v1/gripper.urdf.xacro (robot description, xacro)
@@ -30,6 +30,12 @@
           rpy="0 0 0" />
         <geometry>
-          <mesh
-            filename="package://blue_descriptions/meshes/hand_base_link.STL" />
+          <xacro:if value="${is_gazebo == 'false'}">
+            <mesh
+              filename="package://blue_descriptions/meshes/gripper_full_link.STL" />
+          </xacro:if>
+          <xacro:if value="${is_gazebo}">
+            <mesh
+              filename="package://blue_descriptions/meshes/hand_base_link.STL" />
+          </xacro:if>
         </geometry>
         <material name="">
@@ -42,6 +48,12 @@
           rpy="0 0 0" />
         <geometry>
-          <mesh
-            filename="package://blue_descriptions/meshes/hand_base_link.STL" />
+          <xacro:if value="${is_gazebo == 'false'}">
+            <mesh
+              filename="package://blue_descriptions/meshes/gripper_full_link.STL" />
+          </xacro:if>
+          <xacro:if value="${is_gazebo}">
+            <mesh
+              filename="package://blue_descriptions/meshes/hand_base_link.STL" />
+          </xacro:if>
         </geometry>
       </collision>

Commit message: fixed urdf

File: blue_descriptions/urdf/gripper_v1/gripper.urdf.xacro (robot description, xacro)
@@ -67,7 +67,10 @@
       name="${side}_gripper_finger_joint"
       type="fixed">
+      <!-- <origin -->
+        <!-- xyz="0 0.0 -0.18" -->
+        <!-- rpy="1.5708 1.5708 1.5708" /> -->
       <origin
         xyz="0 0.0 -0.18"
-        rpy="1.5708 1.5708 1.5708" />
+        rpy="-3.14159 -0.0 1.5708" />
       <parent
         link="${side}_${parent}" />

Commit message: removed mass of grippers

File: blue_descriptions/urdf/gripper_v1/gripper.urdf.xacro (robot description, xacro)
@@ -11,18 +11,4 @@
     <link
       name="${side}_${name}">
-      <inertial>
-        <origin
-          xyz="0.00526385736219506 2.70691865020822E-05 -0.0641638075944594"
-          rpy="0 0 0" />
-        <mass
-          value="0.657109755986862" />
-        <inertia
-          ixx="0.0057866591250737"
-          ixy="3.71515699629511E-07"
-          ixz="-6.32890111626103E-05"
-          iyy="0.00530223654324281"
-          iyz="8.9999884666805E-07"
-          izz="0.00342399181200673" />
-      </inertial>
       <visual>
         <origin

Commit message: updates

File: blue_descriptions/urdf/gripper_v1/gripper.urdf.xacro (robot description, xacro)
@@ -15,6 +15,8 @@
           xyz="0.00526385736219506 2.70691865020822E-05 -0.0641638075944594"
           rpy="0 0 0" />
-        <mass
-          value="0.657109755986862" />
+        <!-- <mass -->
+          <!-- value="0.657109755986862" /> -->
+        <mass
+          value="0." />
         <inertia
           ixx="0.0057866591250737"
@@ -84,12 +86,12 @@
           rpy="0 0 0" />
         <mass
-          value="0.0047109755986862" />
-        <inertia
-          ixx="0.000916887873826385"
-          ixy="-6.04547948818479E-08"
-          ixz="0.6796133363069E-06"
-          iyy="0.000877268801166351"
-          iyz="0.64172907801915E-07"
-          izz="0.000293333065172452" />
+          value="0.0" />
+        <inertia
+          ixx="0.0"
+          ixy="0.0"
+          ixz="0.0"
+          iyy="0.0"
+          iyz="0.0"
+          izz="0.0" />
       </inertial>
     </link>
@@ -133,12 +135,12 @@
           rpy="0 0 0" />
         <mass
-          value="0.0384620979765985" />
-        <inertia
-          ixx="1.93716279065148E-05"
-          ixy="-1.74835869619804E-06"
-          ixz="3.21020594362941E-11"
-          iyy="5.23390911087335E-06"
-          iyz="-5.04535602261134E-11"
-          izz="1.92560542157392E-05" />
+          value="0.0" />
+        <inertia
+          ixx="0.0"
+          ixy="0.0"
+          ixz="0.0"
+          iyy="0.0"
+          iyz="0.0"
+          izz="0.0" />
       </inertial>
       <visual>
@@ -189,12 +191,12 @@
           rpy="0 0 0" />
         <mass
-          value="0.0096424502794395" />
-        <inertia
-          ixx="1.76146900164229E-06"
-          ixy="-1.63725174281941E-11"
-          ixz="-5.09403577370148E-07"
-          iyy="1.95368501856251E-06"
-          iyz="-2.7403586363238E-12"
-          izz="6.78506827465793E-07" />
+          value="0.0" />
+        <inertia
+          ixx="0.0"
+          ixy="0.0"
+          ixz="0.0"
+          iyy="0.0"
+          iyz="0.0"
+          izz="0.0" />
       </inertial>
       <visual>
@@ -246,12 +248,12 @@
           rpy="0 0 0" />
         <mass
-          value="0.0384620979765985" />
-        <inertia
-          ixx="1.93716279065148E-05"
-          ixy="-1.74835869619804E-06"
-          ixz="3.21020594362941E-11"
-          iyy="5.23390911087335E-06"
-          iyz="-5.04535602261134E-11"
-          izz="1.92560542157392E-05" />
+          value="0.0" />
+        <inertia
+          ixx="0.0"
+          ixy="0.0"
+          ixz="0.0"
+          iyy="0.0"
+          iyz="0.0"
+          izz="0.0" />
       </inertial>
       <visual>
@@ -302,12 +304,12 @@
           rpy="0 0 0" />
         <mass
-          value="0.0096424502794395" />
-        <inertia
-          ixx="1.76146900164229E-06"
-          ixy="-1.63725174281941E-11"
-          ixz="-5.09403577370148E-07"
-          iyy="1.95368501856251E-06"
-          iyz="-2.7403586363238E-12"
-          izz="6.78506827465793E-07" />
+          value="0.0" />
+        <inertia
+          ixx="0.0"
+          ixy="0.0"
+          ixz="0.0"
+          iyy="0.0"
+          iyz="0.0"
+          izz="0.0" />
       </inertial>
       <visual>

Commit message: Add friction to last link

File: blue_descriptions/urdf/gripper_v1/gripper.urdf.xacro (robot description, xacro)
@@ -344,4 +344,5 @@
       name="${side}_l_finger_tip_joint"
       type="continuous">
+      <dynamics damping="0.7" friction="10.0"/>
       <origin
         xyz="0 0.06 0"

Commit message: Enable mimic joints in gazebo

File: blue_descriptions/urdf/gripper_v1/gripper.urdf.xacro (robot description, xacro)
@@ -8,4 +8,22 @@
     <xacro:blue_gripper_finger_v1 side="${side}" parent="${name}"/>
   </xacro:macro>
+  <xacro:macro name="mimic_joint_plugin_gazebo" params="name_prefix parent_joint mimic_joint has_pid:=false multiplier:=1.0 offset:=0 sensitiveness:=0.0 max_effort:=1.0 robot_namespace:=''">
+    <gazebo>
+      <plugin name="${name_prefix}_mimic_joint_plugin" filename="libroboticsgroup_gazebo_mimic_joint_plugin.so">
+        <joint>${parent_joint}</joint>
+        <mimicJoint>${mimic_joint}</mimicJoint>
+        <xacro:if value="${has_pid}">                     <!-- if set to true, PID parameters from "/gazebo_ros_control/pid_gains/${mimic_joint}" are loaded -->
+          <hasPID />
+        </xacro:if>
+        <multiplier>${multiplier}</multiplier>
+        <offset>${offset}</offset>
+        <sensitiveness>${sensitiveness}</sensitiveness>   <!-- if absolute difference between setpoint and process value is below this threshold, do nothing; 0.0 = disable [rad] -->
+        <maxEffort>${max_effort}</maxEffort>              <!-- only taken into account if has_pid:=true [Nm] -->
+        <xacro:unless value="${robot_namespace == ''}">
+          <robotNamespace>($robot_namespace)</robotNamespace>
+        </xacro:unless>
+      </plugin>
+    </gazebo>
+  </xacro:macro>
   <xacro:macro name="blue_end_v1" params="side name">
     <link
@@ -30,12 +48,6 @@
           rpy="0 0 0" />
         <geometry>
-          <xacro:if value="${is_gazebo == 'false'}">
-            <mesh
-              filename="package://blue_descriptions/meshes/hand_base_link.STL" />
-          </xacro:if>
-          <xacro:if value="${is_gazebo}">
-            <mesh
-              filename="package://blue_descriptions/meshes/gripper_full_link.STL" />
-          </xacro:if>
+          <mesh
+            filename="package://blue_descriptions/meshes/hand_base_link.STL" />
         </geometry>
         <material name="">
@@ -48,12 +60,6 @@
           rpy="0 0 0" />
         <geometry>
-          <xacro:if value="${is_gazebo == 'false'}">
-            <mesh
-              filename="package://blue_descriptions/meshes/hand_base_link.STL" />
-          </xacro:if>
-          <xacro:if value="${is_gazebo}">
-            <mesh
-              filename="package://blue_descriptions/meshes/gripper_full_link.STL" />
-          </xacro:if>
+          <mesh
+            filename="package://blue_descriptions/meshes/hand_base_link.STL" />
         </geometry>
       </collision>
@@ -186,4 +192,7 @@
         multiplier="1"/>
     </joint>
+    <xacro:mimic_joint_plugin_gazebo name_prefix="${side}_r_finger_joint"
+      parent_joint="${side}_gripper_joint" mimic_joint="${side}_r_finger_joint"
+      has_pid="false" multiplier="1.0" max_effort="10.0" />
     <link
       name="${side}_r_finger_tip_link">
@@ -228,5 +237,6 @@
     <joint
       name="${side}_r_finger_tip_joint"
-      type="continuous">
+      type="revolute">
+      <limit lower="0.5" upper="1" velocity="0.7" effort="100" />
         <dynamics damping="0.7" friction="10.0"/>
       <origin
@@ -243,4 +253,7 @@
         multiplier="-1"/>
     </joint>
+    <xacro:mimic_joint_plugin_gazebo name_prefix="${side}_r_finger_tip_joint"
+      parent_joint="${side}_gripper_joint" mimic_joint="${side}_r_finger_tip_joint"
+      has_pid="true" multiplier="-0.25" offset="0.85" max_effort="20" />
     <!-- left finger -->
     <link
@@ -343,5 +356,6 @@
     <joint
       name="${side}_l_finger_tip_joint"
-      type="continuous">
+      type="revolute">
+      <limit lower="0.5" upper="1" velocity="0.7" effort="100" />
       <dynamics damping="0.7" friction="10.0"/>
       <origin
@@ -358,4 +372,7 @@
         multiplier="-1"/>
     </joint>
+    <xacro:mimic_joint_plugin_gazebo name_prefix="${side}_l_finger_tip_joint"
+      parent_joint="${side}_gripper_joint" mimic_joint="${side}_l_finger_tip_joint"
+      has_pid="true" multiplier="-0.25" offset="0.85" max_effort="20" />
     </xacro:if>
   </xacro:macro>

Commit message: Update gripper xacro to allow for mimic joints

File: blue_descriptions/urdf/gripper_v1/gripper.urdf.xacro (robot description, xacro)
@@ -133,5 +133,4 @@
       </transmission>
     </xacro:if>
-    <xacro:if value="${is_gazebo == 'false'}">
     <!-- right finger -->
     <link
@@ -192,7 +191,9 @@
         multiplier="1"/>
     </joint>
-    <xacro:mimic_joint_plugin_gazebo name_prefix="${side}_r_finger_joint"
-      parent_joint="${side}_gripper_joint" mimic_joint="${side}_r_finger_joint"
-      has_pid="false" multiplier="1.0" max_effort="10.0" />
+    <xacro:if value="${is_gazebo}">
+      <xacro:mimic_joint_plugin_gazebo name_prefix="${side}_r_finger_joint"
+        parent_joint="${side}_gripper_joint" mimic_joint="${side}_r_finger_joint"
+        has_pid="false" multiplier="1.0" max_effort="10.0" />
+    </xacro:if>
     <link
       name="${side}_r_finger_tip_link">
@@ -238,9 +239,9 @@
       name="${side}_r_finger_tip_joint"
       type="revolute">
-      <limit lower="0.5" upper="1" velocity="0.7" effort="100" />
+      <limit lower="0.5" upper="1" velocity="0.7" effort="5" />
         <dynamics damping="0.7" friction="10.0"/>
       <origin
         xyz="0 0.06 0"
-        rpy="1.5708 -1.5754E-31 -2.5019" />
+        rpy="1.5708 -1.5754E-31 -3.5019" />
       <parent
         link="${side}_r_finger_link" />
@@ -249,11 +250,15 @@
       <axis
         xyz="0 1 0" />
-      <mimic
-        joint="${side}_gripper_joint"
-        multiplier="-1"/>
-    </joint>
-    <xacro:mimic_joint_plugin_gazebo name_prefix="${side}_r_finger_tip_joint"
-      parent_joint="${side}_gripper_joint" mimic_joint="${side}_r_finger_tip_joint"
-      has_pid="true" multiplier="-0.25" offset="0.85" max_effort="20" />
+        <mimic
+          joint="${side}_gripper_joint"
+          multiplier="-0.25"
+          offset="0.85"
+          max_effort="5"/>
+    </joint>
+    <xacro:if value="${is_gazebo}">
+      <xacro:mimic_joint_plugin_gazebo name_prefix="${side}_r_finger_tip_joint"
+        parent_joint="${side}_gripper_joint" mimic_joint="${side}_r_finger_tip_joint"
+        has_pid="true" multiplier="-0.25" offset="0.85" max_effort="5" />
+    </xacro:if>
     <!-- left finger -->
     <link
@@ -314,4 +319,9 @@
         multiplier="1"/>
     </joint>
+    <xacro:if value="${is_gazebo}">
+      <xacro:mimic_joint_plugin_gazebo name_prefix="${side}_l_finger_joint"
+        parent_joint="${side}_gripper_joint" mimic_joint="${side}_l_finger_joint"
+        has_pid="false" multiplier="1.0" max_effort="10.0" />
+    </xacro:if>
     <link
       name="${side}_l_finger_tip_link">
@@ -357,9 +367,9 @@
       name="${side}_l_finger_tip_joint"
       type="revolute">
-      <limit lower="0.5" upper="1" velocity="0.7" effort="100" />
+      <limit lower="0.5" upper="1" velocity="0.7" effort="5" />
       <dynamics damping="0.7" friction="10.0"/>
       <origin
         xyz="0 0.06 0"
-        rpy="1.5708 -1.5754E-31 -2.5019" />
+        rpy="1.5708 -1.5754E-31 -3.5019" />
       <parent
         link="${side}_l_finger_link" />
@@ -368,11 +378,14 @@
       <axis
         xyz="0 1 0" />
-      <mimic
-        joint="${side}_gripper_joint"
-        multiplier="-1"/>
-    </joint>
-    <xacro:mimic_joint_plugin_gazebo name_prefix="${side}_l_finger_tip_joint"
-      parent_joint="${side}_gripper_joint" mimic_joint="${side}_l_finger_tip_joint"
-      has_pid="true" multiplier="-0.25" offset="0.85" max_effort="20" />
+        <mimic
+          joint="${side}_gripper_joint"
+          multiplier="-0.25"
+          offset="0.85"
+          max_effort="5"/>
+    </joint>
+    <xacro:if value="${is_gazebo}">
+      <xacro:mimic_joint_plugin_gazebo name_prefix="${side}_l_finger_tip_joint"
+        parent_joint="${side}_gripper_joint" mimic_joint="${side}_l_finger_tip_joint"
+        has_pid="true" multiplier="-0.5" offset="0.85" max_effort="5" />
     </xacro:if>
   </xacro:macro>

Commit message: Resolve indentation issue

File: blue_descriptions/urdf/gripper_v1/gripper.urdf.xacro (robot description, xacro)
@@ -104,5 +104,5 @@
       name="${side}_gripper_joint"
       type="revolute">
-        <dynamics damping="0.7" friction="10.0"/>
+      <dynamics damping="0.7" friction="10.0"/>
       <origin
         xyz="0 0 -0.10"

Commit message: Resolve indentation issue

File: blue_descriptions/urdf/gripper_v1/gripper.urdf.xacro (robot description, xacro)
@@ -240,5 +240,5 @@
       type="revolute">
       <limit lower="0.5" upper="1" velocity="0.7" effort="5" />
-        <dynamics damping="0.7" friction="10.0"/>
+      <dynamics damping="0.7" friction="10.0"/>
       <origin
         xyz="0 0.06 0"

Commit message: Fix gripper mimic joint parameters

File: blue_descriptions/urdf/gripper_v1/gripper.urdf.xacro (robot description, xacro)
@@ -238,6 +238,5 @@
     <joint
       name="${side}_r_finger_tip_joint"
-      type="revolute">
-      <limit lower="0.5" upper="1" velocity="0.7" effort="5" />
+      type="continuous">
       <dynamics damping="0.7" friction="10.0"/>
       <origin
@@ -259,5 +258,5 @@
       <xacro:mimic_joint_plugin_gazebo name_prefix="${side}_r_finger_tip_joint"
         parent_joint="${side}_gripper_joint" mimic_joint="${side}_r_finger_tip_joint"
-        has_pid="true" multiplier="-0.25" offset="0.85" max_effort="5" />
+        has_pid="false" multiplier="-1" offset="0" max_effort="0.1" />
     </xacro:if>
     <!-- left finger -->
@@ -366,6 +365,5 @@
     <joint
       name="${side}_l_finger_tip_joint"
-      type="revolute">
-      <limit lower="0.5" upper="1" velocity="0.7" effort="5" />
+      type="continuous">
       <dynamics damping="0.7" friction="10.0"/>
       <origin
@@ -387,5 +385,5 @@
       <xacro:mimic_joint_plugin_gazebo name_prefix="${side}_l_finger_tip_joint"
         parent_joint="${side}_gripper_joint" mimic_joint="${side}_l_finger_tip_joint"
-        has_pid="true" multiplier="-0.5" offset="0.85" max_effort="5" />
+        has_pid="false" multiplier="-1" offset="0" max_effort="0.1" />
     </xacro:if>
   </xacro:macro>
