Commit message: Update gripper xacros

File: blue_descriptions/urdf/gripper_v1/gripper.urdf.xacro (robot description, xacro)
@@ -8,4 +8,22 @@
     <xacro:blue_gripper_finger_v1 side="${side}" parent="${name}"/>
   </xacro:macro>
+  <xacro:macro name="mimic_joint_plugin_gazebo" params="name_prefix parent_joint mimic_joint has_pid:=false multiplier:=1.0 offset:=0 sensitiveness:=0.0 max_effort:=1.0 robot_namespace:=''">
+    <gazebo>
+      <plugin name="${name_prefix}_mimic_joint_plugin" filename="libroboticsgroup_gazebo_mimic_joint_plugin.so">
+        <joint>${parent_joint}</joint>
+        <mimicJoint>${mimic_joint}</mimicJoint>
+        <xacro:if value="${has_pid}">                     <!-- if set to true, PID parameters from "/gazebo_ros_control/pid_gains/${mimic_joint}" are loaded -->
+          <hasPID />
+        </xacro:if>
+        <multiplier>${multiplier}</multiplier>
+        <offset>${offset}</offset>
+        <sensitiveness>${sensitiveness}</sensitiveness>   <!-- if absolute difference between setpoint and process value is below this threshold, do nothing; 0.0 = disable [rad] -->
+        <maxEffort>${max_effort}</maxEffort>              <!-- only taken into account if has_pid:=true [Nm] -->
+        <xacro:unless value="${robot_namespace == ''}">
+          <robotNamespace>($robot_namespace)</robotNamespace>
+        </xacro:unless>
+      </plugin>
+    </gazebo>
+  </xacro:macro>
   <xacro:macro name="blue_end_v1" params="side name">
     <link
@@ -16,5 +34,5 @@
           rpy="0 0 0" />
         <mass
-          value="0.657109755986862" />
+          value="0.687109755986862" />
         <inertia
           ixx="0.0057866591250737"
@@ -30,12 +48,6 @@
           rpy="0 0 0" />
         <geometry>
-          <xacro:if value="${is_gazebo == 'false'}">
-            <mesh
-              filename="package://blue_descriptions/meshes/hand_base_link.STL" />
-          </xacro:if>
-          <xacro:if value="${is_gazebo}">
-            <mesh
-              filename="package://blue_descriptions/meshes/gripper_full_link.STL" />
-          </xacro:if>
+          <mesh
+            filename="package://blue_descriptions/meshes/hand_base_link.STL" />
         </geometry>
         <material name="">
@@ -48,12 +60,6 @@
           rpy="0 0 0" />
         <geometry>
-          <xacro:if value="${is_gazebo == 'false'}">
-            <mesh
-              filename="package://blue_descriptions/meshes/hand_base_link.STL" />
-          </xacro:if>
-          <xacro:if value="${is_gazebo}">
-            <mesh
-              filename="package://blue_descriptions/meshes/gripper_full_link.STL" />
-          </xacro:if>
+          <mesh
+            filename="package://blue_descriptions/meshes/hand_base_link.STL" />
         </geometry>
       </collision>
@@ -67,4 +73,5 @@
       name="${side}_gripper_finger_joint"
       type="fixed">
+      <dynamics damping="0.7" friction="10.0"/>
       <origin
         xyz="0 0.0 -0.18"
@@ -97,4 +104,5 @@
       name="${side}_gripper_joint"
       type="revolute">
+      <dynamics damping="0.7" friction="10.0"/>
       <origin
         xyz="0 0 -0.10"
@@ -116,4 +124,5 @@
         <type>transmission_interface/SimpleTransmission</type>
         <joint name="${side}_gripper_joint">
+        <dynamics damping="0.7" friction="10.0"/>
           <hardwareInterface>hardware_interface/EffortJointInterface</hardwareInterface>
         </joint>
@@ -124,5 +133,4 @@
       </transmission>
     </xacro:if>
-    <xacro:if value="${is_gazebo == 'false'}">
     <!-- right finger -->
     <link
@@ -169,4 +177,5 @@
       name="${side}_r_finger_joint"
       type="continuous">
+      <dynamics damping="0.7" friction="10.0"/>
       <origin
         xyz="0.000 0.030703 -0.071979"
@@ -182,4 +191,9 @@
         multiplier="1"/>
     </joint>
+    <xacro:if value="${is_gazebo}">
+      <xacro:mimic_joint_plugin_gazebo name_prefix="${side}_r_finger_joint"
+        parent_joint="${side}_gripper_joint" mimic_joint="${side}_r_finger_joint"
+        has_pid="false" multiplier="1.0" max_effort="10.0" />
+    </xacro:if>
     <link
       name="${side}_r_finger_tip_link">
@@ -225,4 +239,5 @@
       name="${side}_r_finger_tip_joint"
       type="continuous">
+      <dynamics damping="0.7" friction="10.0"/>
       <origin
         xyz="0 0.06 0"
@@ -236,6 +251,13 @@
       <mimic
         joint="${side}_gripper_joint"
-        multiplier="-1"/>
-    </joint>
+        multiplier="-1"
+        offset="0"
+        max_effort="5"/>
+    </joint>
+    <xacro:if value="${is_gazebo}">
+      <xacro:mimic_joint_plugin_gazebo name_prefix="${side}_r_finger_tip_joint"
+        parent_joint="${side}_gripper_joint" mimic_joint="${side}_r_finger_tip_joint"
+        has_pid="false" multiplier="-1" offset="0" max_effort="0.1" />
+    </xacro:if>
     <!-- left finger -->
     <link
@@ -282,4 +304,5 @@
       name="${side}_l_finger_joint"
       type="continuous">
+      <dynamics damping="0.7" friction="10.0"/>
       <origin
         xyz="0.000 -0.030703 -0.071979"
@@ -295,4 +318,9 @@
         multiplier="1"/>
     </joint>
+    <xacro:if value="${is_gazebo}">
+      <xacro:mimic_joint_plugin_gazebo name_prefix="${side}_l_finger_joint"
+        parent_joint="${side}_gripper_joint" mimic_joint="${side}_l_finger_joint"
+        has_pid="false" multiplier="1.0" max_effort="10.0" />
+    </xacro:if>
     <link
       name="${side}_l_finger_tip_link">
@@ -338,4 +366,5 @@
       name="${side}_l_finger_tip_joint"
       type="continuous">
+      <dynamics damping="0.7" friction="10.0"/>
       <origin
         xyz="0 0.06 0"
@@ -349,6 +378,12 @@
       <mimic
         joint="${side}_gripper_joint"
-        multiplier="-1"/>
-    </joint>
+        multiplier="-1"
+        offset="0"
+        max_effort="5"/>
+    </joint>
+    <xacro:if value="${is_gazebo}">
+      <xacro:mimic_joint_plugin_gazebo name_prefix="${side}_l_finger_tip_joint"
+        parent_joint="${side}_gripper_joint" mimic_joint="${side}_l_finger_tip_joint"
+        has_pid="false" multiplier="-1" offset="0" max_effort="0.1" />
     </xacro:if>
   </xacro:macro>
