Commit message: Make model moveable

File: blue_descriptions/urdf/robot_base_v1/robot_base.urdf.xacro (robot description, xacro)
@@ -4,12 +4,4 @@
   <!-- ============================  Robot Base  ============================ -->
   <xacro:macro name="blue_robot_base_v1" params="cam_height cam_angle is_gazebo:=false">
-  <xacro:if value="${is_gazebo}">
-    <link name="world"/>
-    <joint name ="world_joint" type= "fixed">
-      <origin xyz="0 0 1.4" rpy="0 0 0" />
-      <parent link="world"/>
-      <child link="base_link"/>
-    </joint>
-  </xacro:if>
   <link
     name="base_link">
@@ -42,9 +34,8 @@
     <collision>
       <origin
-        xyz="0 0 0"
+        xyz="0 0 -0.965"
         rpy="0 0 0" />
       <geometry>
-        <mesh
-          filename="package://blue_descriptions/meshes/robot_base_link.STL" />
+        <box size="1 .75 0.001"/>
       </geometry>
     </collision>

Commit message: Add world joint to gazebo

File: blue_descriptions/urdf/robot_base_v1/robot_base.urdf.xacro (robot description, xacro)
@@ -4,4 +4,12 @@
   <!-- ============================  Robot Base  ============================ -->
   <xacro:macro name="blue_robot_base_v1" params="cam_height cam_angle is_gazebo:=false">
+  <xacro:if value="${is_gazebo}">
+    <link name="world"/>
+    <joint name ="world_joint" type= "fixed">
+      <origin xyz="0 0 0.965" rpy="0 0 0" />
+      <parent link="world"/>
+      <child link="base_link"/>
+    </joint>
+  </xacro:if>
   <link
     name="base_link">

Commit message: Remove fixed joint to world in gazebo urdf

File: blue_descriptions/urdf/robot_base_v1/robot_base.urdf.xacro (robot description, xacro)
@@ -4,12 +4,4 @@
   <!-- ============================  Robot Base  ============================ -->
   <xacro:macro name="blue_robot_base_v1" params="cam_height cam_angle is_gazebo:=false">
-  <xacro:if value="${is_gazebo}">
-    <link name="world"/>
-    <joint name ="world_joint" type= "fixed">
-      <origin xyz="0 0 0.965" rpy="0 0 0" />
-      <parent link="world"/>
-      <child link="base_link"/>
-    </joint>
-  </xacro:if>
   <link
     name="base_link">
